File: Switch/new.kicad_sch (KiCad schematic)
At the start: 9 parts, among them J1 RJ45, J2 RJ45, J3 RJ45, J4 RJ45, SW1 Driver/Auton, SW2 Enable/Disable, SW3 Pin7, SW4 Pin4, SW5 Pin1

Commit message: finalize comp switch
Parts:
- J1, J2, J3, J4: footprint RJ45Connector:RJ45-TH_RC0139 -> ghost:RJ45-TH_RC0139
- SW1, SW2, SW3, SW4, SW5: footprint Library:SW-SMD_MS-22D28-G020 -> ghost:SW-SMD_MS-22D28-G020
Changed lines of the file:
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@@
 			)
 		)
-		(property "Footprint" "Library:SW-SMD_MS-22D28-G020"
+		(property "Footprint" "ghost:SW-SMD_MS-22D28-G020"
 			(at 95.25 62.23 0)
 			(effects
@@
 			)
 		)
-		(property "Footprint" "Library:SW-SMD_MS-22D28-G020"
+		(property "Footprint" "ghost:SW-SMD_MS-22D28-G020"
 			(at 95.25 91.44 0)
 			(effects
@@
 			)
 		)
-		(property "Footprint" "RJ45Connector:RJ45-TH_RC0139"
+		(property "Footprint" "ghost:RJ45-TH_RC0139"
 			(at 243.84 130.175 90)
 			(effects
@@
 			)
 		)
-		(property "Footprint" "RJ45Connector:RJ45-TH_RC0139"
+		(property "Footprint" "ghost:RJ45-TH_RC0139"
 			(at 243.84 51.435 90)
 			(effects
@@
 			)
 		)
-		(property "Footprint" "Library:SW-SMD_MS-22D28-G020"
+		(property "Footprint" "ghost:SW-SMD_MS-22D28-G020"
 			(at 99.06 116.84 0)
 			(effects
@@
 			)
 		)
-		(property "Footprint" "RJ45Connector:RJ45-TH_RC0139"
+		(property "Footprint" "ghost:RJ45-TH_RC0139"
 			(at 243.84 103.505 90)
 			(effects
@@
 			)
 		)
-		(property "Footprint" "Library:SW-SMD_MS-22D28-G020"
+		(property "Footprint" "ghost:SW-SMD_MS-22D28-G020"
 			(at 146.05 128.27 0)
 			(effects
@@
 			)
 		)
-		(property "Footprint" "RJ45Connector:RJ45-TH_RC0139"
+		(property "Footprint" "ghost:RJ45-TH_RC0139"
 			(at 243.84 76.835 90)
 			(effects
@@
 			)
 		)
-		(property "Footprint" "Library:SW-SMD_MS-22D28-G020"
+		(property "Footprint" "ghost:SW-SMD_MS-22D28-G020"
 			(at 179.07 148.59 0)
 			(effects
