File: sensor/sensor/sensor.kicad_sch (KiCad schematic)
At the start: 35 parts, among them J1 RJ12_Shielded, J2 Conn_01x04, J3 Conn_01x06, J8 RJ12_Shielded, J9 Conn_01x06, SW5 SW_Coded_SH-7050, U1 PCA9615DP, U2 LTC4316xDD, U5 TPS73101DBV

Commit message: BOM added capacitors
Parts:
- C1: Manufacturer_Part_Number (none) -> 0402B102K500NT; Supplier Part Number (none) -> C1523
- C2, C3: Manufacturer_Part_Number (none) -> CL10A105KB8NNNC; Supplier Part Number (none) -> C15849
- J2: Supplier Part Number C51940130 -> (none); now left out of the parts list
- J3, J9: Supplier Part Number C160405 -> (none); now left out of the parts list
- U1: Manufacturer_Part_Number (none) -> PCA9615DP; Supplier Name JLCPCB -> NXP; now left out of the parts list
- U2: now left out of the parts list
Changed lines of the file:
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@@
 		(unit 1)
 		(exclude_from_sim no)
-		(in_bom yes)
+		(in_bom no)
 		(on_board yes)
 		(dnp no)
@@
 			)
 		)
-		(property "Supplier Part Number" ""
+		(property "Supplier Part Number" "C15849"
+			(at 29.21 173.99 0)
+			(effects
+				(font
+					(size 1.27 1.27)
+				)
+				(hide yes)
+			)
+		)
+		(property "Manufacturer_Part_Number" "CL10A105KB8NNNC"
 			(at 29.21 173.99 0)
 			(effects
@@
 		(unit 1)
 		(exclude_from_sim no)
-		(in_bom yes)
+		(in_bom no)
 		(on_board yes)
 		(dnp no)
@@
 			)
 		)
-		(property "Supplier Part Number" "C160405"
+		(property "Supplier Part Number" ""
 			(at 270.51 77.47 0)
 			(effects
@@
 			)
 		)
-		(property "Supplier Part Number" ""
+		(property "Supplier Part Number" "C15849"
+			(at 83.82 173.99 0)
+			(effects
+				(font
+					(size 1.27 1.27)
+				)
+				(hide yes)
+			)
+		)
+		(property "Manufacturer_Part_Number" "CL10A105KB8NNNC"
 			(at 83.82 173.99 0)
 			(effects
@@
 		(exclude_from_sim no)
 		(in_bom yes)
-		(on_board no)
+		(on_board yes)
 		(dnp no)
 		(fields_autoplaced yes)
@@
 			)
 		)
-		(property "Supplier Part Number" ""
+		(property "Supplier Part Number" "C1523"
+			(at 74.93 173.99 0)
+			(effects
+				(font
+					(size 1.27 1.27)
+				)
+				(hide yes)
+			)
+		)
+		(property "Manufacturer_Part_Number" "0402B102K500NT"
 			(at 74.93 173.99 0)
 			(effects
@@
 		(exclude_from_sim no)
 		(in_bom yes)
-		(on_board no)
+		(on_board yes)
 		(dnp no)
 		(fields_autoplaced yes)
@@
 		(unit 1)
 		(exclude_from_sim no)
-		(in_bom yes)
+		(in_bom no)
 		(on_board yes)
 		(dnp no)
@@
 			)
 		)
-		(property "Supplier Part Number" "C51940130"
+		(property "Supplier Part Number" ""
 			(at 132.08 96.52 0)
 			(effects
@@
 		(unit 1)
 		(exclude_from_sim no)
-		(in_bom yes)
+		(in_bom no)
 		(on_board yes)
 		(dnp no)
@@
 			)
 		)
-		(property "Supplier Part Number" "C160405"
+		(property "Supplier Part Number" ""
 			(at 222.25 139.7 90)
 			(effects
@@
 		(unit 1)
 		(exclude_from_sim no)
-		(in_bom yes)
+		(in_bom no)
 		(on_board yes)
 		(dnp no)
@@
 			)
 		)
-		(property "Supplier Name" "JLCPCB"
+		(property "Supplier Name" "NXP"
 			(at 163.83 77.47 0)
 			(effects
@@
 			(at 163.83 77.47 0)
 			(effects
+				(font
+					(size 1.27 1.27)
+				)
+				(hide yes)
+			)
+		)
+		(property "Manufacturer_Part_Number" "PCA9615DP"
+			(at 163.83 77.47 0)
+			(effects
