File: color+proximity breakout/color+proximity/sensors.kicad_sch (KiCad schematic)
At the start: 24 parts, among them IC1 VL53L4CDV0DH_1, IC2 ISL29125IROZ-T7, U6 ICM-20602

Commit message: not my finest work but at least it works (i hope)
Parts:
- added J4: Conn_01x05, Connector_PinHeader_1.00mm:PinHeader_1x05_P1.00mm_Vertical, symbol Connector_Generic:Conn_01x05
Connections:
- net +3.3V: now also J4.3 (Pin_3)
- net +5V: now also J4.4 (Pin_4)
- net GND: now also J4.5 (Pin_5)
- net scl: now also J4.2 (Pin_2)
- net sda: now also J4.1 (Pin_1)
