File: color+proximity breakout/color+proximity/color+proximity.kicad_sch (KiCad schematic)
At the start: 35 parts, among them J1 RJ12_Shielded, J2 Conn_01x04, J3 Conn_01x06, J8 RJ12_Shielded, J9 Conn_01x06, SW5 SW_Coded_SH-7050, U1 PCA9615DP, U2 LTC4316, U5 TPS73101DBV

Commit message: not my finest work but at least it works (i hope)
Parts:
- removed C1: 1n, Capacitor_SMD:C_0402_1005Metric_Pad0.74x0.62mm_HandSolder, symbol Device:C
- removed C2, C3: 1u, Capacitor_SMD:C_0603_1608Metric_Pad1.08x0.95mm_HandSolder, symbol Device:C
- removed H1, H2: MountingHole_Pad, MountingHole:MountingHole_4.5mm_Pad_TopOnly, symbol Mechanical:MountingHole_Pad
- removed J1, J8: RJ12_Shielded, RJ12_Pin_Connector:RJ12_Pin_Connector, symbol Connector:RJ12_Shielded
- removed J2: Conn_01x04, Connector_JST:JST_SH_SM04B-SRSS-TB_1x04-1MP_P1.00mm_Horizontal, symbol Connector_Generic:Conn_01x04
- removed J3, J9: Conn_01x06, Connector_JST:JST_SH_SM06B-SRSS-TB_1x06-1MP_P1.00mm_Horizontal, symbol Connector_Generic:Conn_01x06
- removed R1, R3, R4, R6: 600, Resistor_SMD:R_0402_1005Metric_Pad0.72x0.64mm_HandSolder, symbol Device:R
- removed R10: 52k, Resistor_SMD:R_0402_1005Metric_Pad0.72x0.64mm_HandSolder, symbol Device:R
- removed R11: 30k, Resistor_SMD:R_0402_1005Metric_Pad0.72x0.64mm_HandSolder, symbol Device:R
- removed R12, R24: 400k, Resistor_SMD:R_0402_1005Metric_Pad0.72x0.64mm_HandSolder, symbol Device:R
- removed R13: 750k, Resistor_SMD:R_0402_1005Metric_Pad0.72x0.64mm_HandSolder, symbol Device:R
- removed R14, R26, R27, R9: 10k, Resistor_SMD:R_0402_1005Metric_Pad0.72x0.64mm_HandSolder, symbol Device:R
- removed R2, R5: 120, Resistor_SMD:R_0402_1005Metric_Pad0.72x0.64mm_HandSolder, symbol Device:R
- removed R25: 780k, Resistor_SMD:R_0402_1005Metric_Pad0.72x0.64mm_HandSolder, symbol Device:R
- removed R28: 80k, Resistor_SMD:R_0402_1005Metric_Pad0.72x0.64mm_HandSolder, symbol Device:R
- removed R29: 40k, Resistor_SMD:R_0402_1005Metric_Pad0.72x0.64mm_HandSolder, symbol Device:R
- removed R31: 260k, Resistor_SMD:R_0402_1005Metric_Pad0.72x0.64mm_HandSolder, symbol Device:R
- removed R7, R8: 4.7k, Resistor_SMD:R_0402_1005Metric_Pad0.72x0.64mm_HandSolder, symbol Device:R
- removed SW5: SW_Coded_SH-7050, RJ12_Pin_Connector:Rotary_Switch_16_pos, symbol Switch:SW_Coded_SH-7050
- removed U1: PCA9615DP, Package_SO:TSSOP-10_3x3mm_P0.5mm, symbol Interface:PCA9615DP
- removed U2: LTC4316, Package_SO:MSOP-10_3x3mm_P0.5mm, symbol Interface_Expansion:LTC4316xDD
- removed U5: TPS73101DBV, Package_TO_SOT_SMD:SOT-23-5, symbol Regulator_Linear:TPS73101DBV
- added C10, C11, C5, C7: 0.1u, Capacitor_SMD:C_0402_1005Metric_Pad0.74x0.62mm_HandSolder, symbol Device:C
- added C12: 4.7u, Capacitor_SMD:C_0603_1608Metric_Pad1.08x0.95mm_HandSolder, symbol Device:C
- added C4: 1u, Capacitor_SMD:C_0603_1608Metric_Pad1.08x0.95mm_HandSolder, symbol Device:C
- added C8: 2.2u, Capacitor_SMD:C_0603_1608Metric_Pad1.08x0.95mm_HandSolder, symbol Device:C
- added C9: 10n, Capacitor_SMD:C_0402_1005Metric_Pad0.74x0.62mm_HandSolder, symbol Device:C
- added D1, D2: WHITE, LED_SMD:LED_0805_2012Metric_Pad1.15x1.40mm_HandSolder, symbol Device:LED
- added IC1: VL53L4CDV0DH_1, VL53L4CD:VL53L4CDV0DH1, symbol VL53L4CDV0DH_1:VL53L4CDV0DH_1
- added IC2: ISL29125IROZ-T7, ISL29125:ISL29125IROZT7, symbol ISL29125:ISL29125IROZ-T7
- added J4: Conn_01x05, Connector_PinHeader_2.54mm:PinHeader_1x05_P2.54mm_Vertical, symbol Connector_Generic:Conn_01x05
- added R15: 100, Resistor_SMD:R_0402_1005Metric_Pad0.72x0.64mm_HandSolder, symbol Device:R
- added R16, R19, R22, R23: 4.7k, Resistor_SMD:R_0402_1005Metric_Pad0.72x0.64mm_HandSolder, symbol Device:R
- added R17, R18, R30, R32: 120, Resistor_SMD:R_0402_1005Metric, symbol Device:R
- added R20, R21: 10k, Resistor_SMD:R_0402_1005Metric_Pad0.72x0.64mm_HandSolder, symbol Device:R
- added U6: ICM-20602, Package_LGA:LGA-16_3x3mm_P0.5mm_LayoutBorder3x5y, symbol Sensor_Motion:ICM-20602
Connections:
- net +3.3V: now also C11.1, C12.1, C7.1, C8.1, C9.1, IC1.1 (AVDDVCSEL_1), IC1.11 (AVDD), IC1.13 (AVDDVCSEL_2), J4.3 (Pin_3), R15.2, R16.1, R19.1, R20.2, R21.1, R22.1, R23.1, U6.1 (VDDIO), U6.16 (VDD)
- net +5V: now also D1.2 (A), D2.2 (A), J4.4 (Pin_4)
- net GND: now also C10.2, C11.2, C12.2, C4.2, C5.2, C7.2, C8.2, C9.2, IC1.12 (GND4), IC1.2 (AVSSVCSEL), IC1.3 (GND), IC1.4 (GND2), IC1.6 (GND3), IC2.3 (GND), J4.5 (Pin_5), R30.2, R32.2, U6.10 (GND), U6.11 (GND), U6.12 (GND), U6.13 (GND), U6.15 (GND), U6.4 (SAO/SD0), U6.8 (FSYNC), U6.9 (GND)
- new net: R18.2, R32.1
- new net: C4.1, C5.1, IC2.1 (VDD), R15.1
- new net: IC2.5 (~{INT}), R16.2
- new net: IC1.7 (GPIO1), R20.1
- new net: D2.1 (K), R18.1
- new net: R17.2, R30.1
- new net: R19.2, U6.5 (~{CS})
- new net: D1.1 (K), R17.1
- new net: C10.1, U6.14 (REGOUT)
- new net: IC1.5 (XSHUT), R21.2
- new net scl: IC1.10 (SCL), IC2.6 (SCL), J4.2 (Pin_2), R23.2, U6.2 (SCL/SPC)
- new net sda: IC1.9 (SDA), IC2.4 (SDA), J4.1 (Pin_1), R22.2, U6.3 (SDA/SDI)
- no-connect marks 3 -> 2
Other:
- removed sheet Sensors
- note added: "Assume 2.9V 8mA, but we can solder over the second set to increase brightness"
- note added: "ICM-20602"
- note added: "ISL29125"
- note added: "Mark specially on silkscreen"
- note added: "VL53L4CD"
- note removed: "For 2.5v R1=40k R2=37k"
- note removed: "For 3.3v R1=52k R2=30k"

Commit message: jOHUGYIFUG#CH@VDJIOwewfurhgvwbdjqnkdiofrguhybfedwqnskjmlidorfguthefdwjqnk2
Parts:
- removed C10, C7: 0.1u, Capacitor_SMD:C_0402_1005Metric_Pad0.74x0.62mm_HandSolder, symbol Device:C
- removed C8: 2.2u, Capacitor_SMD:C_0603_1608Metric_Pad1.08x0.95mm_HandSolder, symbol Device:C
- removed C9: 10n, Capacitor_SMD:C_0402_1005Metric_Pad0.74x0.62mm_HandSolder, symbol Device:C
- removed R19, R22, R23: 4.7k, Resistor_SMD:R_0402_1005Metric_Pad0.72x0.64mm_HandSolder, symbol Device:R
- removed U6: ICM-20602, Package_LGA:LGA-16_3x3mm_P0.5mm_LayoutBorder3x5y, symbol Sensor_Motion:ICM-20602
Connections:
- net +3.3V: now also J4.2 (Pin_2); no longer J4.3 (Pin_3)
- net +5V: now also J4.1 (Pin_1); no longer J4.4 (Pin_4)
- net scl: now also J4.4 (Pin_4); no longer J4.2 (Pin_2)
- net sda: now also J4.3 (Pin_3); no longer J4.1 (Pin_1)
- no-connect marks 2 -> 1
Other:
- note removed: "ICM-20602"

Commit message: i hate git
Parts:
- added C10, C7: 0.1u, Capacitor_SMD:C_0402_1005Metric_Pad0.74x0.62mm_HandSolder, symbol Device:C
- added C8: 2.2u, Capacitor_SMD:C_0603_1608Metric_Pad1.08x0.95mm_HandSolder, symbol Device:C
- added C9: 10n, Capacitor_SMD:C_0402_1005Metric_Pad0.74x0.62mm_HandSolder, symbol Device:C
- added R19: 4.7k, Resistor_SMD:R_0402_1005Metric_Pad0.72x0.64mm_HandSolder, symbol Device:R
- added U6: ICM-20602, Package_LGA:LGA-16_3x3mm_P0.5mm_LayoutBorder3x5y, symbol Sensor_Motion:ICM-20602
Connections:
- net +3.3V: now also C7.1, C8.1, C9.1, R19.1, U6.1 (VDDIO), U6.16 (VDD)
- net GND: now also C10.2, C7.2, C8.2, C9.2, U6.10 (GND), U6.11 (GND), U6.12 (GND), U6.13 (GND), U6.15 (GND), U6.4 (SAO/SD0), U6.8 (FSYNC), U6.9 (GND)
- net scl: now also U6.2 (SCL/SPC)
- net sda: now also U6.3 (SDA/SDI)
- new net: R19.2, U6.5 (~{CS})
- new net: C10.1, U6.14 (REGOUT)
- no-connect marks 1 -> 2
Other:
- note added: "ICM-20602"
