File: solenoid_breakout/solenoid_breakoutboard.kicad_pcb (KiCad board)
At the start: 2 copper layers, 65.5 x 18.5 mm, 27 parts, among them J1 Conn_01x04_Pin, J2 Conn_01x04_Pin, J3 Conn_01x04_Pin, J4 Conn_01x04_Pin, J7 Conn_01x05, J8 Conn_01x05, Q2 AO3400A, Q5 AO3400A, Q6 AO3400A, Q7 AO3400A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

Commit message: small fixes
Connections:
- D2 pad 1: Net-(D2-K) -> +5V
- D3 pad 1: Net-(D3-K) -> +5V
- D4 pad 1: Net-(D4-K) -> +5V
- L2 pad 2: Net-(D2-K) -> +5V
- L3 pad 2: Net-(D3-K) -> +5V
- L4 pad 2: Net-(D4-K) -> +5V
Routing:
- net +5V: track 54.1 -> 64.4 mm
- net Net-(D3-K): track 3.73 -> 0.00 mm
- net Net-(D4-K): track 3.32 -> 0.00 mm
- net Net-(D2-K): track 3.27 -> 0.00 mm
