File: solenoid_breakout/solenoid_breakoutboard.kicad_pcb (KiCad board)
At the start: 2 copper layers, 33.5 x 18.5 mm, 7 parts, among them J1 Conn_01x04_Pin, J2 Conn_01x04_Pin, J3 Conn_01x04_Pin, J4 Conn_01x04_Pin, J7 Conn_01x05, J8 Conn_01x05, U1 PCA9536DP

Commit message: updated base board + updated gpio breakout + added bom/fab files
Parts:
- added G***: LOGO, LOGO, B.Cu at (78.5, 51.8)
- added G***: LOGO, LOGO, B.Cu at (102.0, 52.0)
Routing:
- net +3.3V: track 51.8 -> 51.1 mm
Other:
- board text added: "VEXU GHOST IEEE RAS"
- board text removed: "Property of Ghost Robotics"
- board text removed: "et. al."

Commit message: gpio board iteration 2 updated
Parts:
- removed the J1 at (104.3, 55.5)
- removed the J2 at (99.0, 55.4)
- removed J7, J8: Conn_01x05, Connector_PinHeader_2.54mm:PinHeader_1x05_P2.54mm_Vertical
- added ? (x2): , , F.Cu at (123.5, 64.5)
- added ? (x2): , , F.Cu at (117.2, 51.8)
- added C1: 0.1uF, Capacitor_SMD:C_0402_1005Metric_Pad0.74x0.62mm_HandSolder, F.Cu at (124.5, 57.1)
- added J1: Conn_01x04_Pin, Connector_PinHeader_2.54mm:PinHeader_1x04_P2.54mm_Vertical, F.Cu at (129.5, 53.7)
- added J1: Conn_01x10, pcb_footprints:GT-B0502MSV27-10S1101, F.Cu at (123.5, 51.8)
- added J2: Conn_01x10, pcb_footprints:GT-B0502MSV27-10S1101, F.Cu at (117.2, 64.5)
- added J2: Conn_01x04_Pin, Connector_PinHeader_2.54mm:PinHeader_1x04_P2.54mm_Vertical, F.Cu at (133.5, 53.7)
- moved J4 34.8 mm to (111.0, 53.7)
- moved G*** 32.1 mm to (134.0, 54.4)
- moved G*** 31.6 mm to (110.0, 53.9)
- moved U1 30.3 mm to (120.5, 57.5)
- moved J3 25.5 mm to (107.0, 53.7)
Connections:
- U1 pad 6: scl -> /scl
- U1 pad 7: sda -> /sda
Routing:
- net GND: track 52.2 -> 8.79 mm, vias 3 -> 5
- net scl: track 25.1 -> 0.00 mm, vias 4 -> 0
- net /sda: track 0.00 -> 19.9 mm
- net sda: track 18.9 -> 0.00 mm
- net /scl: track 0.00 -> 14.5 mm
- net Net-(J2-Pin_2): track 17.5 -> 29.6 mm
- net Net-(J3-Pin_2): track 6.87 -> 12.5 mm, vias 1 -> 0
- net Net-(J4-Pin_2): track 13.0 -> 7.74 mm, vias 1 -> 0
- net +5V: track 45.1 -> 40.0 mm, vias 0 -> 3
- net Net-(J1-Pin_2): track 12.9 -> 10.2 mm
- net +3.3V: track 51.1 -> 50.4 mm, vias 2 -> 3
- added copper zone on B.Cu, net GND
Other:
- board size 33.5 x 18.5 mm -> 31.5 x 20 mm
- board text added: "Designed by Lakshay Yadav Trung Le"
- board text removed: "Designed by Lakshay Yadav"

Commit message: breakout board iteration 2 updates
Parts:
- removed the ? at (123.5, 64.5)
- removed the ? at (117.2, 51.8)
- moved G*** 4.60 mm to (131.5, 50.5)
- moved G*** 3.51 mm to (109.0, 50.5)
Routing:
- net GND: track 8.79 -> 9.88 mm
- net +5V: track 40.0 -> 39.5 mm

Commit message: gpio iteration 2 update
Parts:
- added C2: 10uF, Capacitor_SMD:C_0402_1005Metric_Pad0.74x0.62mm_HandSolder, F.Cu at (127.0, 54.0)
- added C3: 10uF, Capacitor_SMD:C_0402_1005Metric_Pad0.74x0.62mm_HandSolder, F.Cu at (113.5, 64.5)
Routing:
- net +3.3V: track 50.4 -> 53.7 mm

Commit message: updated production files
Parts:
- G*** (x2): moved to F.Cu
- J5: renamed from J2; moved to B.Cu
- J6: renamed from J1; moved to B.Cu
- U1: value PCA9536DP -> TCA9536DTMR
- moved G*** 28.7 mm to (107.0, 65.4), turned to 0 degrees
- moved G*** 15.1 mm to (110.7, 65.5), turned to 0 degrees
- turned J5 to 0 degrees
- turned J6 to 180 degrees
Connections:
- J5 pad 10: +5V -> GND
- J5 pad 6: GND -> +5V
- J5 pad 7: /scl -> +3.3V
- J5 pad 9: +3.3V -> /scl
- J6 pad 10: +5V -> GND
- J6 pad 6: GND -> +5V
- J6 pad 7: /scl -> +3.3V
- J6 pad 9: +3.3V -> /scl
Routing:
- net +3.3V: track 53.7 -> 58.7 mm, vias 3 -> 2
- net GND: track 9.88 -> 5.23 mm
- net +5V: track 39.5 -> 38.4 mm, vias 3 -> 1
- net /sda: track 19.9 -> 20.8 mm, vias 0 -> 2
- net /scl: track 14.5 -> 14.6 mm, vias 0 -> 2
Other:
- board text added: "Designed by: Lakshay Yadav Trung Le"
- board text removed: "Designed by Lakshay Yadav Trung Le"
