File: sensor_base/sensor.kicad_sch (KiCad schematic)
At the start: 35 parts, among them IC1 LTC4316CMS, J1 GDLX-SMT-N-66, J2 Conn_01x04, J3 Conn_01x06, J6 GDLX-SMT-N-66, J9 Conn_01x06, SW5 SW_Coded_SH-7050, U1 PCA9615DP, U5 TPS73101DBV

Commit message: finished rtc schematic
Parts:
- SW5: footprint RJ12_Pin_Connector:Rotary_Switch_16_pos -> pcb_footprints:Rotary_Switch_16_pos
Changed lines of the file:
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@@
 			)
 		)
-		(property "Footprint" "RJ12_Pin_Connector:Rotary_Switch_16_pos"
+		(property "Footprint" "pcb_footprints:Rotary_Switch_16_pos"
 			(at 17.78 140.97 0)
 			(effects
