File: sensor_base/sensor.kicad_pcb (KiCad board)
At the start: 2 copper layers, 66.1 x 19 mm, 42 parts, among them IC1 LTC4316CMS#TRPBF, J1 GDLX-SMT-N-66, J2 Conn_01x04, J3 Conn_01x06, J4 Conn_01x05, J5 Conn_01x05, J6 GDLX-SMT-N-66, J9 Conn_01x06, SW5 SW_Coded_SH-7050, U1 PCA9615DP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

Commit message: updated base board + updated gpio breakout + added bom/fab files
Parts:
- removed the G*** at (110.3, 105.6)
- removed the G*** at (110.7, 102.8)
- added G***: LOGO, GDLX-SMT-N-66:vexu_ghost, F.Cu at (109.7, 107.1)
- added G***: LOGO, LOGO, B.Cu at (149.6, 102.8)
- moved G*** 4.92 mm to (119.7, 102.3), turned to 180 degrees
- moved H1 0.30 mm to (124.2, 109.0)
- moved H2 0.30 mm to (147.1, 109.0)
Other:
- board text added: "3V3"
- board text added: "5V"
- board text added: "ALLEN A KARMANYAAH M"
- board text added: "ANDREW K JENNY C"
- board text added: "GND"
- board text added: "IEEE RAS VEXU GHOST BASE DELOYMENT BOARD"
- board text added: "SCL"
- board text added: "SDA"
- board text removed: "ALLEN A KARMA. M ANDREW K JENNY C"
- board text removed: "IEEE RAS VEXU GHOST SENSOR BOARD"
