File: sensor_base/sensor_base_iteration_2/sensors.kicad_sch (KiCad schematic)
At the start: 4 parts, among them J4 Conn_01x05, J5 Conn_01x05

Commit message: finished base board interation 2 schematic and started on pcb layout
Parts:
- removed J4, J5: Conn_01x05, Connector_PinHeader_2.54mm:PinHeader_1x05_P2.54mm_Vertical, symbol Connector_Generic:Conn_01x05
- added H1, H2: MountingHole, pcb_footprints:MountingHole_#4_3.175mm, symbol Mechanical:MountingHole
- added J4, J5: Conn_02x05_Top_Bottom, pcb_footprints:GT-B0502FSV43-10S1101, symbol Connector_Generic:Conn_02x05_Top_Bottom
Connections:
- net +3.3V: now also J4.2 (Pin_2), J5.2 (Pin_2)
- net +5V: now also J4.1 (Pin_1), J5.1 (Pin_1)
- net GND: now also J4.5 (Pin_5), J5.5 (Pin_5)
- net scl: now also J4.4 (Pin_4), J5.4 (Pin_4)
- net sda: now also J4.3 (Pin_3), J5.3 (Pin_3)
- no-connect marks 0 -> 10
Other:
- note added: "MOUNTING HOLES FOR SENSORS MODULES"

Commit message: finished base board PCB + created production files for base board and modules
Parts:
- J4, J5: Manufacturer_Name (none) -> G-Switch; Manufacturer_Part_Number (none) -> GT-B0502FSV43-10S1101
Changed lines of the file:
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@@
+			)
+		)
+		(property "Manufacturer_Name" "G-Switch"
+			(at 125.73 86.36 0)
+			(effects
+				(font
+					(size 1.27 1.27)
+				)
+				(hide yes)
+			)
+		)
+		(property "Manufacturer_Part_Number" "GT-B0502FSV43-10S1101"
+			(at 125.73 86.36 0)
+			(effects
+				(font
+					(size 1.27 1.27)
+				)
+				(hide yes)
 			)
 		)
@@
 			(at 152.4 86.36 0)
 			(effects
+				(font
+					(size 1.27 1.27)
+				)
+				(hide yes)
+			)
+		)
+		(property "Manufacturer_Name" "G-Switch"
+			(at 152.4 86.36 0)
+			(effects
+				(font
+					(size 1.27 1.27)
+				)
+				(hide yes)
+			)
+		)
+		(property "Manufacturer_Part_Number" "GT-B0502FSV43-10S1101"
+			(at 152.4 86.36 0)
+			(effects
