File: sensor_base/sensor_base_iteration_2/sensor_base_iteration_2.kicad_sch (KiCad schematic)
At the start: 49 parts, among them IC1 LTC4316CMS, J1 GDLX-SMT-N-66, J2 Conn_01x04, J3 Conn_01x06, J6 GDLX-SMT-N-66, J9 Conn_01x06, SW5 SW_Coded_SH-7050, U1 PCA9615DP, U5 TPS73101DBV

Commit message: finished base board interation 2 schematic and started on pcb layout
Parts:
- removed H1, H2: MountingHole_Pad, MountingHole:MountingHole_4.5mm_Pad_TopOnly, symbol Mechanical:MountingHole_Pad
- removed J1, J6: GDLX-SMT-N-66, GDLX-SMT-N-66:GDLXSMTN66, symbol GDLX-SMT-N-66:GDLX-SMT-N-66
- removed R10: 52k, Resistor_SMD:R_0402_1005Metric_Pad0.72x0.64mm_HandSolder, symbol Device:R
- removed R11: 30k, Resistor_SMD:R_0402_1005Metric_Pad0.72x0.64mm_HandSolder, symbol Device:R
- removed TP1, TP10, TP11, TP12, TP13, TP2, TP3, TP4, TP5, TP6, TP7, TP8, TP9: TestPoint, symbol Connector:TestPoint
- removed U5: TPS73101DBV, Package_TO_SOT_SMD:SOT-23-5, symbol Regulator_Linear:TPS73101DBV
- added H3, H4, H5, H6: MountingHole, pcb_footprints:MountingHole_#4_3.175mm, symbol Mechanical:MountingHole
- added J1, J6: Conn_01x04, Connector_PinHeader_1.27mm:PinHeader_1x04_P1.27mm_Vertical, symbol Connector_Generic:Conn_01x04
- added J7: Conn_01x03, Connector_PinHeader_1.27mm:PinHeader_1x03_P1.27mm_Vertical, symbol Connector_Generic:Conn_01x03
- added J8: Conn_01x02, Connector_PinHeader_1.27mm:PinHeader_1x02_P1.27mm_Vertical, symbol Connector_Generic:Conn_01x02
- added U2: TPS73133DBV, Package_TO_SOT_SMD:SOT-23-5, symbol Regulator_Linear:TPS73133DBV
- C1: value 1n -> 10n
- J2: footprint Connector_JST:JST_SH_SM04B-SRSS-TB_1x04-1MP_P1.00mm_Horizontal -> Connector_JST:JST_GH_SM04B-GHS-TB_1x04-1MP_P1.25mm_Horizontal
- J3, J9: footprint Connector_JST:JST_SH_SM06B-SRSS-TB_1x06-1MP_P1.00mm_Horizontal -> Connector_JST:JST_GH_SM06B-GHS-TB_1x06-1MP_P1.25mm_Horizontal
- SW5: Manufacturer_Part_Number ES07MP-16RBZ-L1500 -> ES07MH-16RBZ-L1000; Supplier Part Number (none) -> C50395976
Connections:
- net +3.3V: now also J7.2 (Pin_2), U2.5 (OUT); no longer C1.1
- net +5V: now also J9.6 (Pin_6), J7.1 (Pin_1), U2.1 (IN), U2.3 (EN); no longer J9.1 (Pin_1)
- net DSCL+: now also J9.3 (Pin_3), J1.3 (Pin_3); no longer J9.4 (Pin_4)
- net DSCL-: now also J9.2 (Pin_2), J1.4 (Pin_4); no longer J9.5 (Pin_5)
- net DSDA+: now also J3.3 (Pin_3), J9.4 (Pin_4), J1.1 (Pin_1); no longer J3.2 (Pin_2), J9.2 (Pin_2)
- net DSDA-: now also J3.2 (Pin_2), J9.5 (Pin_5), J1.2 (Pin_2); no longer J3.3 (Pin_3), J9.3 (Pin_3)
- net GND: now also C1.2, J9.1 (Pin_1), J7.3 (Pin_3), U2.2 (GND); no longer J9.6 (Pin_6)
- net SCLIN: now also J6.1 (Pin_1)
- net SCLOUT: now also J6.3 (Pin_3)
- net SDAIN: now also J6.2 (Pin_2)
- net SDAOUT: now also J6.4 (Pin_4)
- net XORH: now also J8.1 (Pin_1)
- net XORL: now also J8.2 (Pin_2)
- new net: C1.1, U2.4 (NR)
- no-connect marks 3 -> 1
Other:
- moved on the sheet: C1, J2, J3, J9, R1, R2, R3, R4, R5, R6, R7, R8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

Commit message: finished base board PCB + created production files for base board and modules
Parts:
- C1: Manufacturer_Name (none) -> Samsung Electro-Mechanics; Manufacturer_Part_Number (none) -> CL05B103KB5NNNC
- C2, C3: Manufacturer_Name (none) -> Samsung Electro-Mechanics; Manufacturer_Part_Number (none) -> CL10B105KB8NQNC
- C4: Manufacturer_Name (none) -> Samsung Electro-Mechanics; Manufacturer_Part_Number (none) -> CL10A106KP8NNNC
- J1, J6, J7, J8: now left out of the parts list
- J2: Manufacturer_Name (none) -> XYECONN; Manufacturer_Part_Number XY-SM04B-SRSS-TB -> XY-SM04B-GHS-TB
- J3, J9: Manufacturer_Name (none) -> XYECONN; Manufacturer_Part_Number SM06B-SRSS-TB(LF)(SN) -> XY-SM06B-GHS-TB
- U2: Manufacturer_Name (none) -> Texas Instruments; Manufacturer_Part_Number (none) -> TPS73133DBVR
Changed lines of the file:
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@@
 			)
 		)
+		(property "Manufacturer_Name" "Samsung Electro-Mechanics"
+			(at 29.21 177.8 0)
+			(effects
+				(font
+					(size 1.27 1.27)
+				)
+				(hide yes)
+			)
+		)
+		(property "Manufacturer_Part_Number" "CL10B105KB8NQNC"
+			(at 29.21 177.8 0)
+			(effects
+				(font
+					(size 1.27 1.27)
+				)
+				(hide yes)
+			)
+		)
 		(pin "2"
 		)
@@
 			)
 		)
-		(property "Manufacturer_Part_Number" "SM06B-SRSS-TB(LF)(SN)"
+		(property "Manufacturer_Part_Number" "XY-SM06B-GHS-TB"
 			(at 257.81 102.87 0)
 			(effects
@@
 			)
 		)
+		(property "Manufacturer_Name" "XYECONN"
+			(at 257.81 102.87 0)
+			(effects
+				(font
+					(size 1.27 1.27)
+				)
+				(hide yes)
+			)
+		)
 		(pin "6"
 		)
@@
 			)
 		)
+		(property "Manufacturer_Name" "Texas Instruments"
+			(at 46.99 172.72 0)
+			(effects
+				(font
+					(size 1.27 1.27)
+				)
+				(hide yes)
+			)
+		)
+		(property "Manufacturer_Part_Number" "TPS73133DBVR"
+			(at 46.99 172.72 0)
+			(effects
+				(font
+					(size 1.27 1.27)
+				)
+				(hide yes)
+			)
+		)
 		(pin "3"
 		)
@@
 			)
 		)
+		(property "Manufacturer_Name" "Samsung Electro-Mechanics"
+			(at 83.82 173.99 0)
+			(effects
+				(font
+					(size 1.27 1.27)
+				)
+				(hide yes)
+			)
+		)
+		(property "Manufacturer_Part_Number" "CL10B105KB8NQNC"
+			(at 83.82 173.99 0)
+			(effects
+				(font
+					(size 1.27 1.27)
+				)
+				(hide yes)
+			)
+		)
 		(pin "1"
 		)
@@
 		(unit 1)
 		(exclude_from_sim no)
-		(in_bom yes)
+		(in_bom no)
 		(on_board yes)
 		(dnp no)
@@
 			)
 		)
+		(property "Manufacturer_Name" "Samsung Electro-Mechanics"
+			(at 71.12 177.8 0)
+			(effects
+				(font
+					(size 1.27 1.27)
+				)
+				(hide yes)
+			)
+		)
+		(property "Manufacturer_Part_Number" "CL05B103KB5NNNC"
+			(at 71.12 177.8 0)
+			(effects
+				(font
+					(size 1.27 1.27)
+				)
+				(hide yes)
+			)
+		)
 		(pin "1"
 		)
@@
 			)
 		)
-		(property "Manufacturer_Part_Number" "XY-SM04B-SRSS-TB"
+		(property "Manufacturer_Part_Number" "XY-SM04B-GHS-TB"
 			(at 142.24 133.35 0)
 			(effects
@@
 			)
 		)
+		(property "Manufacturer_Name" "XYECONN"
+			(at 142.24 133.35 90)
+			(effects
+				(font
+					(size 1.27 1.27)
+				)
+				(hide yes)
+			)
+		)
 		(pin "4"
 		)
@@
 		(unit 1)
 		(exclude_from_sim no)
-		(in_bom yes)
+		(in_bom no)
 		(on_board yes)
 		(dnp no)
@@
 			)
 		)
+		(property "Manufacturer_Name" "Samsung Electro-Mechanics"
+			(at 19.05 177.8 0)
+			(effects
+				(font
+					(size 1.27 1.27)
+				)
+				(hide yes)
+			)
+		)
+		(property "Manufacturer_Part_Number" "CL10A106KP8NNNC"
+			(at 19.05 177.8 0)
+			(effects
+				(font
+					(size 1.27 1.27)
+				)
+				(hide yes)
+			)
+		)
 		(pin "2"
 		)
@@
 			)
 		)
-		(property "Manufacturer_Part_Number" "SM06B-SRSS-TB(LF)(SN)"
+		(property "Manufacturer_Part_Number" "XY-SM06B-GHS-TB"
 			(at 257.81 134.62 90)
 			(effects
@@
 			)
 		)
+		(property "Manufacturer_Name" "XYECONN"
+			(at 257.81 134.62 90)
+			(effects
+				(font
+					(size 1.27 1.27)
+				)
+				(hide yes)
+			)
+		)
 		(pin "6"
 		)
@@
 		(unit 1)
 		(exclude_from_sim no)
-		(in_bom yes)
+		(in_bom no)
 		(on_board yes)
 		(dnp no)
@@
 		(unit 1)
 		(exclude_from_sim no)
-		(in_bom yes)
+		(in_bom no)
 		(on_board yes)
 		(dnp no)

Commit message: finish host board v2 layout + production files
Parts:
- U1: Manufacturer_Name NXP -> NXP Semiconductors
Changed lines of the file:
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@@
 			)
 		)
-		(property "Manufacturer_Name" "NXP"
+		(property "Manufacturer_Name" "NXP Semiconductors"
 			(at 173.99 102.87 0)
 			(effects
