File: host/ghost_host.kicad_sch (KiCad schematic)
At the start: 11 parts, among them J1 RGB_3_Pin_Connector, U9 kb2040

Commit message: please fix everything
Parts:
- D1: footprint Diode_SMD:D_SOD-323_HandSoldering -> Diode_SMD:D_SOD-128
Connections:
- net GND: no longer H1.1, H2.1, H3.1, H4.1, H5.1, H6.1
Changed lines of the file:
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@@
 	(paper "A4")
 	(junction
-		(at 153.67 25.4)
-		(diameter 0)
-		(color 0 0 0 0)
-	)
-	(junction
-		(at 146.05 25.4)
-		(diameter 0)
-		(color 0 0 0 0)
-	)
-	(junction
 		(at 116.84 72.39)
 		(diameter 0)
@@
 	)
 	(junction
-		(at 142.24 25.4)
-		(diameter 0)
-		(color 0 0 0 0)
-	)
-	(junction
-		(at 137.16 25.4)
-		(diameter 0)
-		(color 0 0 0 0)
-	)
-	(junction
-		(at 161.29 25.4)
-		(diameter 0)
-		(color 0 0 0 0)
-	)
-	(junction
 		(at 116.84 87.63)
 		(diameter 0)
@@
 	(wire
 		(pts
-			(xy 142.24 25.4) (xy 146.05 25.4)
-		)
-		(stroke
-			(width 0)
-			(type default)
-		)
-	)
-	(wire
-		(pts
-			(xy 142.24 25.4) (xy 142.24 26.67)
-		)
-		(stroke
-			(width 0)
-			(type default)
-		)
-	)
-	(wire
-		(pts
 			(xy 68.58 57.15) (xy 68.58 58.42)
 		)
@@
 	(wire
 		(pts
-			(xy 146.05 25.4) (xy 153.67 25.4)
-		)
-		(stroke
-			(width 0)
-			(type default)
-		)
-	)
-	(wire
-		(pts
 			(xy 95.25 52.07) (xy 93.98 52.07)
 		)
@@
 	(wire
 		(pts
-			(xy 153.67 25.4) (xy 161.29 25.4)
-		)
-		(stroke
-			(width 0)
-			(type default)
-		)
-	)
-	(wire
-		(pts
-			(xy 137.16 25.4) (xy 142.24 25.4)
-		)
-		(stroke
-			(width 0)
-			(type default)
-		)
-	)
-	(wire
-		(pts
-			(xy 161.29 25.4) (xy 168.91 25.4)
-		)
-		(stroke
-			(width 0)
-			(type default)
-		)
-	)
-	(wire
-		(pts
-			(xy 129.54 25.4) (xy 137.16 25.4)
-		)
-		(stroke
-			(width 0)
-			(type default)
-		)
-	)
-	(wire
-		(pts
 			(xy 142.24 82.55) (xy 138.43 82.55)
 		)
@@
 			)
 		)
-		(property "Footprint" "Diode_SMD:D_SOD-323_HandSoldering"
+		(property "Footprint" "Diode_SMD:D_SOD-128"
 			(at 91.44 52.07 0)
 			(effects
@@
 					(unit 1)
 				)
-			)
-		)
-	)
-	(symbol
-		(lib_id "power:GND")
-		(at 142.24 26.67 0)
-		(unit 1)
-		(exclude_from_sim no)
-		(in_bom yes)
-		(on_board yes)
-		(dnp no)
-		(fields_autoplaced yes)
-		(property "Reference" "#PWR047"
-			(at 142.24 33.02 0)
-			(effects
-				(font
-					(size 1.27 1.27)
-				)
-				(hide yes)
-			)
-		)
-		(property "Value" "GND"
-			(at 142.24 31.75 0)
-			(effects
-				(font
-					(size 1.27 1.27)
-				)
-			)
-		)
-		(property "Footprint" ""
-			(at 142.24 26.67 0)
-			(effects
-				(font
-					(size 1.27 1.27)
-				)
-				(hide yes)
-			)
-		)
-		(property "Datasheet" ""
-			(at 142.24 26.67 0)
-			(effects
-				(font
-					(size 1.27 1.27)
-				)
-				(hide yes)
-			)
-		)
-		(property "Description" "Power symbol creates a global label with name \"GND\" , ground"
-			(at 142.24 26.67 0)
-			(effects
-				(font
-					(size 1.27 1.27)
-				)
-				(hide yes)
-			)
-		)
-		(pin "1"
-		)
-		(instances
-			(project "ghost_host"
-				(path "/d931a957-36f8-4ac4-bfa7-9b0a51712375"
-					(reference "#PWR047")
-					(unit 1)
-				)

Commit message: started host board layout v2
Parts:
- U9: footprint kb2040:kb2040 -> pcb_footprints:kb2040
Connections:
- no-connect marks 4 -> 10
