File: host/input.kicad_sch (KiCad schematic)
At the start: 15 parts, among them J2 Conn_01x04, J23 RJ12_Shielded, J24 Conn_01x06, U1 PCA9615DP

Commit message: please fix everything
Parts:
- removed J23: RJ12_Shielded, RJ12_Pin_Connector:RJ12_Pin_Connector, symbol Connector:RJ12_Shielded
- added C17: 10uf, Capacitor_SMD:C_0603_1608Metric, symbol Device:C
- added J4: Conn_01x06, Connector_JST:JST_GH_SM06B-GHS-TB_1x06-1MP_P1.25mm_Horizontal, symbol Connector_Generic:Conn_01x06
- added SCL2, SDA2, TP17, TP18, TP33, TP34: TestPoint, TestPoint:TestPoint_Pad_D1.0mm, symbol Connector:TestPoint
- J2: footprint RJ12_Pin_Connector:JST_SH_BM04B-SRSS-TB_1x04-1MP_P1.00mm_Vertical -> Connector_JST:JST_GH_BM04B-GHS-TBT_1x04-1MP_P1.25mm_Vertical
- J24: footprint RJ12_Pin_Connector:JST_SH_BM06B-SRSS-TB_1x06-1MP_P1.00mm_Vertical -> Connector_JST:JST_GH_BM06B-GHS-TBT_1x06-1MP_P1.25mm_Vertical
Connections:
- net 5v: no longer C9.1, J24.1 (Pin_1), R15.1, R9.1, U1.10 (V_{DD(B)})
- net GND: now also C17.2, J4.6 (Pin_6)
- net scl: now also SCL2.1
- net sda: now also SDA2.1
- net at R11.1, R9.2: no longer J24.4 (Pin_4), U1.7 (DSCLP)
- net at R15.2, R65.1, U1.8 (DSDAP): now also J24.3 (Pin_3), J4.3 (Pin_3), TP17.1; no longer J24.2 (Pin_2)
- net at R65.2, R66.1, U1.9 (DSDAM): now also J24.2 (Pin_2), J4.2 (Pin_2), TP18.1; no longer J24.3 (Pin_3)
- net at J24.5 (Pin_5), U1.6 (DSCLM): now also J4.5 (Pin_5), TP34.1
- net 3.3v renamed +3.3V
- new net: J24.4 (Pin_4), J4.4 (Pin_4), TP33.1, U1.7 (DSCLP)
- new net +5V: C17.1, C9.1, J24.1 (Pin_1), J4.1 (Pin_1), R15.1, R9.1, U1.10 (V_{DD(B)})
Other:
- note added: "swtitch 2 and 3"
- moved on the sheet: C1, C9, J2, J24, R1, R11, R13, R15, R2, R65, R66, R7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

Commit message: started host board layout v2
Parts:
- renumbered TP33 to DSCL+5, TP34 to DSCL-5, TP17 to DSDA+5, TP18 to DSDA-5, SCL2 to SCL5, SDA2 to SDA5
Connections:
- net +5V is gone; now on net 5v: C17.1, C9.1, J24.1 (Pin_1), J4.1 (Pin_1), R15.1, R9.1, U1.10 (V_{DD(B)})
- net DSCL-: now reaches R11.2, R13.1
- net DSCL-: now also DSCL-5.1, J24.5 (Pin_5), J4.5 (Pin_5), U1.6 (DSCLM)
- net DSCL+: now reaches R11.1, R9.2
- net DSCL+: now also DSCL+5.1, J24.4 (Pin_4), J4.4 (Pin_4), U1.7 (DSCLP)
- net DSDA-: now reaches DSDA-5.1, J24.2 (Pin_2), J4.2 (Pin_2), R65.2, R66.1, U1.9 (DSDAM)
- net DSDA+: now reaches DSDA+5.1, J24.3 (Pin_3), J4.3 (Pin_3), R15.2, R65.1, U1.8 (DSDAP)
- net +3.3V renamed 3.3v
Other:
- moved on the sheet: DSCL-5, DSDA+5, DSDA-5, J2, R1, R11, R13, R2, R65, R66, R7, R9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
