File: host/ghost_host.kicad_pcb (KiCad board)
At the start: 2 copper layers, 127.5 x 68.5 mm, 133 parts, among them J1 RGB_3_Pin_Connector, J10 Conn_01x06, J11 Conn_01x04, J12 RJ12_Shielded, J13 Conn_01x06, J14 Conn_01x04, J15 RJ12_Shielded, J16 Conn_01x06, J17 Conn_01x04, J18 RJ12_Shielded, J19 Conn_01x06, J2 Conn_01x04, J20 Conn_01x04, J21 RJ12_Shielded, J22 Conn_01x06, J23 RJ12_Shielded, J24 Conn_01x06, J25 Conn_01x06, J3 Conn_01x04, J4 RJ12_Shielded, J5 Conn_01x04, J6 RJ12_Shielded, J7 Conn_01x06, J8 Conn_01x04, J9 RJ12_Shielded, U1 PCA9615DP, U2 PCA9615DP, U3 PCA9615DP, U4 PCA9615DP, U5 PCA9615DP, U6 PCA9615DP, U7 PCA9615DP, U8 PCA9615DP, U9 kb2040

Commit message: please fix everything
Parts:
- added C17: 10uf, Capacitor_SMD:C_0603_1608Metric, F.Cu at (103.1, 69.0)
- added C18: 10uf, Capacitor_SMD:C_0603_1608Metric, F.Cu at (163.0, 106.2)
- added C19: 10uf, Capacitor_SMD:C_0603_1608Metric, F.Cu at (178.9, 69.7)
- added C20: 10uf, Capacitor_SMD:C_0603_1608Metric, F.Cu at (187.8, 104.8)
- added C21: 10uf, Capacitor_SMD:C_0603_1608Metric, F.Cu at (112.2, 106.7)
- added C22: 10uf, Capacitor_SMD:C_0603_1608Metric, F.Cu at (128.2, 70.0)
- added C23: 10uf, Capacitor_SMD:C_0603_1608Metric, F.Cu at (153.6, 70.2)
- added C24: 10uf, Capacitor_SMD:C_0603_1608Metric, F.Cu at (137.6, 107.0)
- added DSCLM2: TestPoint, TestPoint:TestPoint_Pad_D1.0mm, F.Cu at (185.4, 106.4)
- added DSCLP2: TestPoint, TestPoint:TestPoint_Pad_D1.0mm, F.Cu at (183.5, 109.5)
- added DSDAM1: TestPoint, TestPoint:TestPoint_Pad_D1.0mm, F.Cu at (261.4, 133.3)
- added DSDAM2: TestPoint, TestPoint:TestPoint_Pad_D1.0mm, F.Cu at (176.6, 106.0)
- added DSDAP1: TestPoint, TestPoint:TestPoint_Pad_D1.0mm, F.Cu at (261.4, 136.3)
- added DSDAP2: TestPoint, TestPoint:TestPoint_Pad_D1.0mm, F.Cu at (180.6, 106.7)
- added J23: Conn_01x06, Connector_JST:JST_GH_SM06B-GHS-TB_1x06-1MP_P1.25mm_Horizontal, F.Cu at (158.7, 116.0)
- added SCL1: TestPoint, TestPoint:TestPoint_Pad_D1.0mm, F.Cu at (264.4, 133.3)
- added SCL2: TestPoint, TestPoint:TestPoint_Pad_D1.0mm, F.Cu at (258.4, 125.2)
- added SCL3: TestPoint, TestPoint:TestPoint_Pad_D1.0mm, F.Cu at (192.7, 106.3)
- added SDA1: TestPoint, TestPoint:TestPoint_Pad_D1.0mm, F.Cu at (264.4, 136.3)
- added SDA2: TestPoint, TestPoint:TestPoint_Pad_D1.0mm, F.Cu at (258.4, 128.2)
- added SDA3: TestPoint, TestPoint:TestPoint_Pad_D1.0mm, F.Cu at (192.8, 102.8)
- added TP10: TestPoint, TestPoint:TestPoint_Pad_D1.0mm, F.Cu at (232.7, 92.7)
- added TP11: TestPoint, TestPoint:TestPoint_Pad_D1.0mm, F.Cu at (232.7, 76.5)
- added TP12: TestPoint, TestPoint:TestPoint_Pad_D1.0mm, F.Cu at (247.2, 136.3)
- added TP13: TestPoint, TestPoint:TestPoint_Pad_D1.0mm, F.Cu at (232.7, 100.8)
- added TP14: TestPoint, TestPoint:TestPoint_Pad_D1.0mm, F.Cu at (232.7, 84.5)
- added TP17: TestPoint, TestPoint:TestPoint_Pad_D1.0mm, F.Cu at (261.4, 125.2)
- added TP18: TestPoint, TestPoint:TestPoint_Pad_D1.0mm, F.Cu at (261.4, 128.2)
- added TP19: TestPoint, TestPoint:TestPoint_Pad_D1.0mm, F.Cu at (235.8, 89.6)
- added TP2: TestPoint, TestPoint:TestPoint_Pad_D1.0mm, F.Cu at (232.7, 89.6)
- added TP20: TestPoint, TestPoint:TestPoint_Pad_D1.0mm, F.Cu at (235.8, 92.7)
- added TP21: TestPoint, TestPoint:TestPoint_Pad_D1.0mm, F.Cu at (235.8, 73.4)
- added TP22: TestPoint, TestPoint:TestPoint_Pad_D1.0mm, F.Cu at (235.8, 76.5)
- added TP23: TestPoint, TestPoint:TestPoint_Pad_D1.0mm, F.Cu at (250.2, 133.3)
- added TP25: TestPoint, TestPoint:TestPoint_Pad_D1.0mm, F.Cu at (235.8, 97.7)
- added TP26: TestPoint, RJ12_Pin_Connector:JST_SH_BM06B-SRSS-TB_1x06-1MP_P1.00mm_Vertical, F.Cu at (235.8, 100.8)
- added TP27: TestPoint, TestPoint:TestPoint_Pad_D1.0mm, F.Cu at (235.8, 81.5)
- added TP28: TestPoint, TestPoint:TestPoint_Pad_D1.0mm, F.Cu at (235.8, 84.5)
- added TP3: TestPoint, TestPoint:TestPoint_Pad_D1.0mm, F.Cu at (232.7, 73.4)
- added TP33: TestPoint, TestPoint:TestPoint_Pad_D1.0mm, F.Cu at (264.4, 125.2)
- added TP34: TestPoint, TestPoint:TestPoint_Pad_D1.0mm, F.Cu at (264.4, 128.2)
- added TP35: TestPoint, TestPoint:TestPoint_Pad_D1.0mm, F.Cu at (238.8, 89.6)
- added TP36: TestPoint, TestPoint:TestPoint_Pad_D1.0mm, F.Cu at (238.8, 92.7)
- added TP37: TestPoint, TestPoint:TestPoint_Pad_D1.0mm, F.Cu at (238.8, 73.4)
- added TP38: TestPoint, TestPoint:TestPoint_Pad_D1.0mm, F.Cu at (238.8, 76.5)
- added TP39: TestPoint, TestPoint:TestPoint_Pad_D1.0mm, F.Cu at (253.3, 133.3)
- added TP4: TestPoint, TestPoint:TestPoint_Pad_D1.0mm, F.Cu at (247.2, 133.3)
- added TP40: TestPoint, TestPoint:TestPoint_Pad_D1.0mm, F.Cu at (253.3, 136.3)
- added TP41: TestPoint, TestPoint:TestPoint_Pad_D1.0mm, F.Cu at (238.8, 97.7)
- added TP42: TestPoint, TestPoint:TestPoint_Pad_D1.0mm, F.Cu at (238.8, 100.8)
- added TP43: TestPoint, TestPoint:TestPoint_Pad_D1.0mm, F.Cu at (238.8, 81.5)
- added TP44: TestPoint, TestPoint:TestPoint_Pad_D1.0mm, F.Cu at (238.8, 84.5)
- added TP5: TestPoint, TestPoint:TestPoint_Pad_D1.0mm, F.Cu at (232.7, 97.7)
- added TP6: TestPoint, TestPoint:TestPoint_Pad_D1.0mm, F.Cu at (232.7, 81.5)
- D1: footprint Diode_SMD:D_SOD-323_HandSoldering -> Diode_SMD:D_SOD-128
- J10, J13, J19, J22, J24, J25, J7: footprint RJ12_Pin_Connector:JST_SH_BM06B-SRSS-TB_1x06-1MP_P1.00mm_Vertical -> Connector_JST:JST_GH_BM06B-GHS-TBT_1x06-1MP_P1.25mm_Vertical
- J11, J17, J2, J20, J3, J5, J8: footprint RJ12_Pin_Connector:JST_SH_BM04B-SRSS-TB_1x04-1MP_P1.00mm_Vertical -> Connector_JST:JST_GH_BM04B-GHS-TBT_1x04-1MP_P1.25mm_Vertical
- J12, J15, J18, J21, J4, J6, J9: value RJ12_Shielded -> Conn_01x06; footprint RJ12_Pin_Connector:RJ12_Pin_Connector -> Connector_JST:JST_GH_SM06B-GHS-TB_1x06-1MP_P1.25mm_Horizontal
- moved J15 96.4 mm to (143.5, 156.5), turned to 0 degrees
- moved J18 96.0 mm to (107.5, 48.5)
- moved J12 90.3 mm to (188.1, 41.0)
- moved J4 71.5 mm to (105.2, 130.6), turned to 0 degrees
- moved J9 34.3 mm to (158.8, 45.8), turned to 0 degrees
- moved J6 32.4 mm to (136.1, 45.4), turned to 0 degrees
- moved J21 29.2 mm to (184.1, 116.0)
- moved J25 2.10 mm to (137.9, 78.2), turned to 0 degrees
- moved C10 1.93 mm to (121.8, 65.5), turned to 90 degrees
- moved C2 1.55 mm to (119.5, 69.7)
- moved J20 0.47 mm to (164.2, 100.2)
- moved J17 0.24 mm to (189.3, 100.2)
- moved J19 0.21 mm to (178.2, 100.2)
Connections:
- H1 pad 1: GND -> unconnected-(H1-Pad1)
- H2 pad 1: GND -> unconnected-(H2-Pad1)
- H3 pad 1: GND -> unconnected-(H3-Pad1)
- H4 pad 1: GND -> unconnected-(H4-Pad1)
- H5 pad 1: GND -> unconnected-(H5-Pad1)
- H6 pad 1: GND -> unconnected-(H6-Pad1)
- J12 pad 2: Net-(J13-Pin_2) -> Net-(J10-Pin_2)
- J12 pad 3: Net-(J13-Pin_3) -> Net-(J10-Pin_3)
- J12 pad 4: Net-(J13-Pin_4) -> Net-(J10-Pin_4)
- J12 pad 5: Net-(J13-Pin_5) -> Net-(J10-Pin_5)
- J15 pad 2: Net-(J16-Pin_2) -> Net-(J13-Pin_2)
- J15 pad 3: Net-(J16-Pin_3) -> Net-(J13-Pin_3)
- J15 pad 4: Net-(J16-Pin_4) -> Net-(J13-Pin_4)
- J15 pad 5: Net-(J16-Pin_5) -> Net-(J13-Pin_5)
- J18 pad 2: Net-(J19-Pin_2) -> Net-(J16-Pin_2)
- J18 pad 3: Net-(J19-Pin_3) -> Net-(J16-Pin_3)
- J18 pad 4: Net-(J19-Pin_4) -> Net-(J16-Pin_4)
- J18 pad 5: Net-(J19-Pin_5) -> Net-(J16-Pin_5)
- J21 pad 2: Net-(J22-Pin_2) -> Net-(J19-Pin_2)
- J21 pad 3: Net-(J22-Pin_3) -> Net-(J19-Pin_3)
- J21 pad 4: Net-(J22-Pin_4) -> Net-(J19-Pin_4)
- J21 pad 5: Net-(J22-Pin_5) -> Net-(J19-Pin_5)
- J4 pad 2: Net-(J25-Pin_2) -> Net-(J24-Pin_2)
- J4 pad 3: Net-(J25-Pin_3) -> Net-(J24-Pin_3)
- J4 pad 4: Net-(J25-Pin_4) -> Net-(J24-Pin_4)
- J4 pad 5: Net-(J25-Pin_5) -> Net-(J24-Pin_5)
- J6 pad 2: Net-(J7-Pin_2) -> Net-(J25-Pin_2)
- J6 pad 3: Net-(J7-Pin_3) -> Net-(J25-Pin_3)
- J6 pad 4: Net-(J7-Pin_4) -> Net-(J25-Pin_4)
- J6 pad 5: Net-(J7-Pin_5) -> Net-(J25-Pin_5)
- J9 pad 2: Net-(J10-Pin_2) -> Net-(J7-Pin_2)
- J9 pad 3: Net-(J10-Pin_3) -> Net-(J7-Pin_3)
- J9 pad 4: Net-(J10-Pin_4) -> Net-(J7-Pin_4)
- J9 pad 5: Net-(J10-Pin_5) -> Net-(J7-Pin_5)
- R11 pad 1: Net-(J24-Pin_4) -> Net-(R11-Pad1)
- R14 pad 2: Net-(J10-Pin_4) -> Net-(R14-Pad2)
- R15 pad 2: Net-(J24-Pin_2) -> Net-(J24-Pin_3)
- R19 pad 2: Net-(J7-Pin_4) -> Net-(R19-Pad2)
- R20 pad 1: Net-(J7-Pin_4) -> Net-(R19-Pad2)
- R22 pad 2: Net-(J7-Pin_2) -> Net-(J7-Pin_3)
- R23 pad 1: Net-(J7-Pin_2) -> Net-(J7-Pin_3)
- R23 pad 2: Net-(J7-Pin_3) -> Net-(J7-Pin_2)
- R24 pad 1: Net-(J7-Pin_3) -> Net-(J7-Pin_2)
- R25 pad 1: Net-(J10-Pin_4) -> Net-(R14-Pad2)
- R27 pad 1: Net-(J10-Pin_2) -> Net-(J10-Pin_3)
- R27 pad 2: Net-(J10-Pin_3) -> Net-(J10-Pin_2)
- R28 pad 1: Net-(J10-Pin_3) -> Net-(J10-Pin_2)
- R3 pad 2: Net-(J10-Pin_2) -> Net-(J10-Pin_3)
- R32 pad 2: Net-(J13-Pin_4) -> Net-(R32-Pad2)
- R33 pad 1: Net-(J13-Pin_4) -> Net-(R32-Pad2)
- R35 pad 2: Net-(J13-Pin_2) -> Net-(J13-Pin_3)
- R36 pad 1: Net-(J13-Pin_2) -> Net-(J13-Pin_3)
- R36 pad 2: Net-(J13-Pin_3) -> Net-(J13-Pin_2)
- R37 pad 1: Net-(J13-Pin_3) -> Net-(J13-Pin_2)
- R41 pad 2: Net-(J16-Pin_4) -> Net-(R41-Pad2)
- R42 pad 1: Net-(J16-Pin_4) -> Net-(R41-Pad2)
- R44 pad 2: Net-(J16-Pin_2) -> Net-(J16-Pin_3)
- R45 pad 1: Net-(J16-Pin_2) -> Net-(J16-Pin_3)
- R45 pad 2: Net-(J16-Pin_3) -> Net-(J16-Pin_2)
- R46 pad 1: Net-(J16-Pin_3) -> Net-(J16-Pin_2)
- R50 pad 2: Net-(J19-Pin_4) -> Net-(R50-Pad2)
- R51 pad 1: Net-(J19-Pin_4) -> Net-(R50-Pad2)
- R53 pad 2: Net-(J19-Pin_2) -> Net-(J19-Pin_3)
- R54 pad 1: Net-(J19-Pin_2) -> Net-(J19-Pin_3)
- R54 pad 2: Net-(J19-Pin_3) -> Net-(J19-Pin_2)
- R55 pad 1: Net-(J19-Pin_3) -> Net-(J19-Pin_2)
- R59 pad 2: Net-(J22-Pin_4) -> Net-(R59-Pad2)
- R60 pad 1: Net-(J22-Pin_4) -> Net-(R59-Pad2)
- R62 pad 2: Net-(J22-Pin_2) -> Net-(J22-Pin_3)
- R63 pad 1: Net-(J22-Pin_2) -> Net-(J22-Pin_3)
- R63 pad 2: Net-(J22-Pin_3) -> Net-(J22-Pin_2)
- R64 pad 1: Net-(J22-Pin_3) -> Net-(J22-Pin_2)
- R65 pad 1: Net-(J24-Pin_2) -> Net-(J24-Pin_3)
- R65 pad 2: Net-(J24-Pin_3) -> Net-(J24-Pin_2)
- R66 pad 1: Net-(J24-Pin_3) -> Net-(J24-Pin_2)
- R67 pad 2: Net-(J25-Pin_4) -> Net-(R67-Pad2)
- R68 pad 1: Net-(J25-Pin_4) -> Net-(R67-Pad2)
- R70 pad 2: Net-(J25-Pin_2) -> Net-(J25-Pin_3)
- R71 pad 1: Net-(J25-Pin_2) -> Net-(J25-Pin_3)
- R71 pad 2: Net-(J25-Pin_3) -> Net-(J25-Pin_2)
- R72 pad 1: Net-(J25-Pin_3) -> Net-(J25-Pin_2)
- R9 pad 2: Net-(J24-Pin_4) -> Net-(R11-Pad1)
- U1 pad 8: Net-(J24-Pin_2) -> Net-(J24-Pin_3)
- U1 pad 9: Net-(J24-Pin_3) -> Net-(J24-Pin_2)
- U2 pad 8: Net-(J25-Pin_2) -> Net-(J25-Pin_3)
- U2 pad 9: Net-(J25-Pin_3) -> Net-(J25-Pin_2)
- U3 pad 8: Net-(J7-Pin_2) -> Net-(J7-Pin_3)
- U3 pad 9: Net-(J7-Pin_3) -> Net-(J7-Pin_2)
- U4 pad 8: Net-(J10-Pin_2) -> Net-(J10-Pin_3)
- U4 pad 9: Net-(J10-Pin_3) -> Net-(J10-Pin_2)
- U5 pad 8: Net-(J13-Pin_2) -> Net-(J13-Pin_3)
- U5 pad 9: Net-(J13-Pin_3) -> Net-(J13-Pin_2)
- U6 pad 8: Net-(J16-Pin_2) -> Net-(J16-Pin_3)
- U6 pad 9: Net-(J16-Pin_3) -> Net-(J16-Pin_2)
- U7 pad 8: Net-(J19-Pin_2) -> Net-(J19-Pin_3)
- U7 pad 9: Net-(J19-Pin_3) -> Net-(J19-Pin_2)
- U8 pad 8: Net-(J22-Pin_2) -> Net-(J22-Pin_3)
- U8 pad 9: Net-(J22-Pin_3) -> Net-(J22-Pin_2)
Routing:
- net GND: track 461.4 -> 336.7 mm, vias 15 -> 14
- net (no net): track 0.00 -> 88.8 mm
- net Net-(J22-Pin_3): track 17.7 -> 37.2 mm
- net +5V: track 177.8 -> 195.1 mm, vias 16 -> 18
- net Net-(J19-Pin_3): track 17.7 -> 34.9 mm
- net unconnected-(J9-PadSH): track 14.8 -> 0.00 mm
- net unconnected-(J6-PadSH): track 14.8 -> 0.00 mm
- net unconnected-(J4-PadSH): track 14.8 -> 0.00 mm
- net unconnected-(J23-PadSH): track 14.8 -> 0.00 mm
- net unconnected-(J21-PadSH): track 14.8 -> 0.00 mm
- net unconnected-(J18-PadSH): track 14.8 -> 0.00 mm
- net unconnected-(J15-PadSH): track 14.8 -> 0.00 mm
- net unconnected-(J12-PadSH): track 14.8 -> 0.00 mm
- net Net-(J22-Pin_5): track 14.3 -> 21.3 mm, vias 0 -> 1
- net Net-(J25-Pin_3): track 17.7 -> 24.6 mm
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
Commit message: started host board layout v2
Parts:
- removed C1, C11, C12, C13, C15, C16, C3, C4, C5, C7, C8, C9: 1u, Capacitor_SMD:C_0603_1608Metric
- removed C17, C19, C20, C21, C23, C24: 10uf, Capacitor_SMD:C_0603_1608Metric
- removed DSCLM2, DSCLP2, DSDAM1, DSDAM2, DSDAP1, DSDAP2, SCL3, SDA3, TP10, TP11, TP12, TP13, TP17, TP18, TP19, TP2, TP20, TP21, TP22, TP23, TP25, TP3, TP33, TP34, TP35, TP36, TP37, TP38, TP39, TP4, TP40, TP41, TP42, TP5: TestPoint, TestPoint:TestPoint_Pad_D1.0mm
- removed J10, J13, J19, J22, J24, J25, J7: Conn_01x06, Connector_JST:JST_GH_BM06B-GHS-TBT_1x06-1MP_P1.25mm_Vertical
- removed J11, J17, J2, J20, J3, J5, J8: Conn_01x04, Connector_JST:JST_GH_BM04B-GHS-TBT_1x04-1MP_P1.25mm_Vertical
- removed J12, J15, J21, J23, J4, J9: Conn_01x06, Connector_JST:JST_GH_SM06B-GHS-TB_1x06-1MP_P1.25mm_Horizontal
- removed J16: Conn_01x06, RJ12_Pin_Connector:JST_SH_BM06B-SRSS-TB_1x06-1MP_P1.00mm_Vertical
- removed J23: RJ12_Shielded, RJ12_Pin_Connector:RJ12_Pin_Connector
- removed R1, R10, R16, R17, R2, R29, R30, R47, R48, R56, R57, R8: 4.7k, Resistor_SMD:R_0603_1608Metric_Pad0.98x0.95mm_HandSolder
- removed R11, R20, R23, R25, R27, R33, R36, R51, R54, R60, R63, R65: 120, Resistor_SMD:R_0603_1608Metric_Pad0.98x0.95mm_HandSolder
- removed R12, R18, R31, R49, R58, R7: 10k, Resistor_SMD:R_0603_1608Metric_Pad0.98x0.95mm_HandSolder
- removed R13, R14, R15, R19, R21, R22, R24, R26, R28, R3, R32, R34, R35, R37, R50, R52, R53, R55, R59, R61, R62, R64, R66, R9: 600, Resistor_SMD:R_0603_1608Metric_Pad0.98x0.95mm_HandSolder
- removed the SCL1 at (264.4, 133.3)
- removed the SDA1 at (264.4, 136.3)
- removed TP26: TestPoint, RJ12_Pin_Connector:JST_SH_BM06B-SRSS-TB_1x06-1MP_P1.00mm_Vertical
- removed U1, U3, U4, U5, U7, U8: PCA9615DP, Package_SO:TSSOP-10_3x3mm_P0.5mm
- added DSCL+2: TestPoint, TestPoint:TestPoint_Pad_D1.0mm, F.Cu at (140.4, 55.5)
- added DSCL-2: TestPoint, TestPoint:TestPoint_Pad_D1.0mm, F.Cu at (140.4, 57.5)
- added DSDA+2: TestPoint, TestPoint:TestPoint_Pad_D1.0mm, F.Cu at (125.9, 55.5)
- added DSDA-2: TestPoint, TestPoint:TestPoint_Pad_D1.0mm, F.Cu at (125.9, 57.5)
- added REF**: TestPoint, TestPoint:TestPoint_Pad_D1.0mm, F.Cu at (83.9, 21.3)
- added REF**: Conn_01x04, Connector_JST:JST_GH_BM04B-GHS-TBT_1x04-1MP_P1.25mm_Vertical, F.Cu at (133.2, 74.4)
- added REF**: 600, Resistor_SMD:R_0603_1608Metric_Pad0.98x0.95mm_HandSolder, B.Cu at (99.2, 35.3)
- added REF**: 600, Resistor_SMD:R_0603_1608Metric_Pad0.98x0.95mm_HandSolder, B.Cu at (85.5, 35.1)
- added REF**: 600, Resistor_SMD:R_0603_1608Metric_Pad0.98x0.95mm_HandSolder, B.Cu at (95.6, 35.3)
- added REF**: 1u, Capacitor_SMD:C_0603_1608Metric, B.Cu at (100.9, 35.3)
- added REF**: 600, Resistor_SMD:R_0603_1608Metric_Pad0.98x0.95mm_HandSolder, B.Cu at (81.9, 35.2)
- added REF**: 1u, Capacitor_SMD:C_0603_1608Metric, B.Cu at (79.9, 35.0)
- added REF**: 120, Resistor_SMD:R_0603_1608Metric_Pad0.98x0.95mm_HandSolder, B.Cu at (97.4, 35.3)
- added REF**: PCA9615DP, Package_SO:TSSOP-10_3x3mm_P0.5mm, B.Cu at (90.5, 35.8)
- added REF**: 120, Resistor_SMD:R_0603_1608Metric_Pad0.98x0.95mm_HandSolder, B.Cu at (83.7, 35.1)
- added REF**: TestPoint, TestPoint:TestPoint_Pad_D1.0mm, F.Cu at (98.4, 21.3)
- added REF**: 10uf, Capacitor_SMD:C_0603_1608Metric, B.Cu at (78.2, 35.0)
- added REF**: Conn_01x06, Connector_JST:JST_GH_SM06B-GHS-TB_1x06-1MP_P1.25mm_Horizontal, B.Cu at (91.2, 23.0)
- added REF**: 4.7k, Resistor_SMD:R_0603_1608Metric_Pad0.98x0.95mm_HandSolder, F.Cu at (89.7, 27.6)
- added REF**: TestPoint, TestPoint:TestPoint_Pad_D1.0mm, F.Cu at (93.4, 28.7)
- added REF**: 4.7k, Resistor_SMD:R_0603_1608Metric_Pad0.98x0.95mm_HandSolder, F.Cu at (89.7, 29.2)
- added REF**: TestPoint, TestPoint:TestPoint_Pad_D1.0mm, F.Cu at (83.9, 23.3)
- added REF**: 10k, Resistor_SMD:R_0603_1608Metric_Pad0.98x0.95mm_HandSolder, F.Cu at (89.7, 30.8)
- added REF**: TestPoint, TestPoint:TestPoint_Pad_D1.0mm, F.Cu at (96.3, 30.7)
- added REF**: TestPoint, TestPoint:TestPoint_Pad_D1.0mm, F.Cu at (98.4, 23.3)
- C18, C22, J18, J6: moved to B.Cu
- J14: footprint RJ12_Pin_Connector:JST_SH_BM04B-SRSS-TB_1x04-1MP_P1.00mm_Vertical -> Connector_JST:JST_GH_BM04B-GHS-TBT_1x04-1MP_P1.25mm_Vertical
- R38, R39, R4, R40, R5, R6: moved to F.Cu
- U9: footprint kb2040:kb2040 -> pcb_footprints:kb2040
- moved SDA2 139.3 mm to (135.4, 62.9)
- moved DSDA-1 137.9 mm to (100.5, 57.5)
- moved DSDA+1 137.7 mm to (100.5, 55.5)
- moved SCL2 134.4 mm to (138.3, 64.9)
- moved DSCL-1 126.7 mm to (115.0, 57.5)
- moved DSCL+1 126.5 mm to (115.0, 55.5)
- moved SDA1 124.6 mm to (110.0, 62.9)
- moved SCL1 121.0 mm to (112.8, 64.8)
- moved C18 56.6 mm to (120.2, 69.2), turned to 90 degrees
- moved C22 33.4 mm to (94.8, 69.2), turned to 90 degrees
- moved C2 23.5 mm to (142.9, 69.5)
- moved C6 23.0 mm to (117.5, 69.5), turned to 90 degrees
- moved C14 21.3 mm to (96.5, 69.2)
- moved R67 15.3 mm to (141.2, 69.5), turned to -90 degrees
- moved R41 15.3 mm to (115.8, 69.5), turned to -90 degrees
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- renumbered TP43 to DSCL+1, TP44 to DSCL-1, TP27 to DSDA+1, TP28 to DSDA-1, TP6 to SCL1, TP14 to SDA1
Connections:
- net Net-(J16-Pin_2) renamed /input5/DSDA-
- net Net-(J16-Pin_3) renamed /input5/DSDA+
- net Net-(J25-Pin_2) renamed /input1/DSDA-
- net Net-(J25-Pin_3) renamed /input1/DSDA+
- DSCL+1 pad 1: Net-(J16-Pin_4) -> /input5/DSCL+
- DSCL-1 pad 1: Net-(J16-Pin_5) -> /input5/DSCL-
- J18 pad 4: Net-(J16-Pin_4) -> /input5/DSCL+
- J18 pad 5: Net-(J16-Pin_5) -> /input5/DSCL-
- J6 pad 4: Net-(J25-Pin_4) -> /input1/DSCL+
- J6 pad 5: Net-(J25-Pin_5) -> /input1/DSCL-
- R41 pad 2: Net-(R41-Pad2) -> /input5/DSCL+
- R42 pad 1: Net-(R41-Pad2) -> /input5/DSCL+
- R42 pad 2: Net-(R42-Pad2) -> /input5/DSCL-
- R43 pad 1: Net-(R42-Pad2) -> /input5/DSCL-
- R67 pad 2: Net-(R67-Pad2) -> /input1/DSCL+
- R68 pad 1: Net-(R67-Pad2) -> /input1/DSCL+
- R68 pad 2: Net-(R68-Pad2) -> /input1/DSCL-
- R69 pad 1: Net-(R68-Pad2) -> /input1/DSCL-
- SCL2 pad 1: /scl5 -> /scl3
- SDA2 pad 1: /sda5 -> /sda3
- U2 pad 6: Net-(J25-Pin_5) -> /input1/DSCL-
- U2 pad 7: Net-(J25-Pin_4) -> /input1/DSCL+
- U6 pad 6: Net-(J16-Pin_5) -> /input5/DSCL-
- U6 pad 7: Net-(J16-Pin_4) -> /input5/DSCL+
Routing:
- net GND: track 336.7 -> 120.9 mm, vias 14 -> 9
- net (no net): track 88.8 -> 3.43 mm
- net /input5/DSCL+: track 0.00 -> 74.9 mm, vias 0 -> 2
- net /input5/DSCL-: track 0.00 -> 74.8 mm, vias 0 -> 2
- net /input5/DSDA+: track 17.0 -> 78.5 mm, vias 1 -> 2
- net /input5/DSDA-: track 24.6 -> 74.9 mm, vias 1 -> 2
- net /input1/DSCL+: track 0.00 -> 37.4 mm, vias 0 -> 1
- net /input1/DSCL-: track 0.00 -> 37.4 mm, vias 0 -> 1
- net Net-(J22-Pin_3): track 37.2 -> 0.00 mm, vias 1 -> 0
- net Net-(J19-Pin_3): track 34.9 -> 0.00 mm, vias 1 -> 0
- net /scl6: track 37.6 -> 2.77 mm, vias 3 -> 0
- net /sda2: track 15.8 -> 49.6 mm, vias 1 -> 3
- net /scl2: track 24.2 -> 57.2 mm, vias 1 -> 3
- net /scl3: track 22.3 -> 53.6 mm, vias 2 -> 3
- net Net-(J22-Pin_4): track 30.6 -> 0.00 mm, vias 1 -> 0
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Other:
- board text removed: "Input 3"
- board text removed: "Input 4"
- board text removed: "Input 5"
- board text removed: "Input 6"
- board text removed: "Input 7"
- board text removed: "Input 8"

Commit message: host board updated
Parts:
- added C1: 1u, Capacitor_SMD:C_0603_1608Metric, B.Cu at (98.1, 119.9)
- added C11: 1u, Capacitor_SMD:C_0603_1608Metric, B.Cu at (147.3, 69.2)
- added C12: 1u, Capacitor_SMD:C_0603_1608Metric, B.Cu at (172.6, 69.2)
- added C13: 1u, Capacitor_SMD:C_0603_1608Metric, B.Cu at (144.6, 107.1)
- added C15: 1u, Capacitor_SMD:C_0603_1608Metric, B.Cu at (195.4, 110.2)
- added C16: 1u, Capacitor_SMD:C_0603_1608Metric, B.Cu at (169.9, 107.1)
- added C17: 10uf, Capacitor_SMD:C_0603_1608Metric, B.Cu at (120.8, 107.1)
- added C19: 10uf, Capacitor_SMD:C_0603_1608Metric, B.Cu at (145.6, 69.2)
- added C20: 10uf, Capacitor_SMD:C_0603_1608Metric, B.Cu at (170.9, 69.2)
- added C21: 10uf, Capacitor_SMD:C_0603_1608Metric, B.Cu at (146.2, 107.1)
- added C23: 10uf, Capacitor_SMD:C_0603_1608Metric, B.Cu at (195.4, 114.2)
- added C24: 10uf, Capacitor_SMD:C_0603_1608Metric, B.Cu at (171.6, 107.1)
- added C3: 1u, Capacitor_SMD:C_0603_1608Metric, B.Cu at (168.3, 69.5)
- added C4: 1u, Capacitor_SMD:C_0603_1608Metric, B.Cu at (193.7, 69.5)
- added C5: 1u, Capacitor_SMD:C_0603_1608Metric, B.Cu at (123.5, 106.8)
- added C7: 1u, Capacitor_SMD:C_0603_1608Metric, B.Cu at (174.3, 106.9)
- added C8: 1u, Capacitor_SMD:C_0603_1608Metric, B.Cu at (148.9, 106.8)
- added C9: 1u, Capacitor_SMD:C_0603_1608Metric, B.Cu at (119.2, 107.1)
- added DSCL+3: TestPoint, TestPoint:TestPoint_Pad_D1.0mm, F.Cu at (165.8, 55.5)
- added DSCL+4: TestPoint, TestPoint:TestPoint_Pad_D1.0mm, F.Cu at (191.2, 55.5)
- added DSCL+5: TestPoint, TestPoint:TestPoint_Pad_D1.0mm, F.Cu at (100.6, 120.8)
- added DSCL+6: TestPoint, TestPoint:TestPoint_Pad_D1.0mm, F.Cu at (126.0, 120.8)
- added DSCL+7: TestPoint, TestPoint:TestPoint_Pad_D1.0mm, F.Cu at (151.4, 120.8)
- added DSCL+8: TestPoint, TestPoint:TestPoint_Pad_D1.0mm, F.Cu at (176.8, 120.9)
- added DSCL-3: TestPoint, TestPoint:TestPoint_Pad_D1.0mm, F.Cu at (165.8, 57.5)
- added DSCL-4: TestPoint, TestPoint:TestPoint_Pad_D1.0mm, F.Cu at (191.2, 57.5)
- added DSCL-5: TestPoint, TestPoint:TestPoint_Pad_D1.0mm, F.Cu at (100.6, 118.8)
- added DSCL-6: TestPoint, TestPoint:TestPoint_Pad_D1.0mm, F.Cu at (126.0, 118.8)
- added DSCL-7: TestPoint, TestPoint:TestPoint_Pad_D1.0mm, F.Cu at (151.4, 118.8)
- added DSCL-8: TestPoint, TestPoint:TestPoint_Pad_D1.0mm, F.Cu at (176.8, 118.9)
- added DSDA+3: TestPoint, TestPoint:TestPoint_Pad_D1.0mm, F.Cu at (151.3, 55.5)
- added DSDA+4: TestPoint, TestPoint:TestPoint_Pad_D1.0mm, F.Cu at (176.7, 55.5)
- added DSDA+5: TestPoint, TestPoint:TestPoint_Pad_D1.0mm, F.Cu at (115.1, 120.8)
- added DSDA+6: TestPoint, TestPoint:TestPoint_Pad_D1.0mm, F.Cu at (140.5, 120.8)
- added DSDA+7: TestPoint, TestPoint:TestPoint_Pad_D1.0mm, F.Cu at (165.9, 120.8)
- added DSDA+8: TestPoint, TestPoint:TestPoint_Pad_D1.0mm, F.Cu at (191.3, 120.9)
- added DSDA-3: TestPoint, TestPoint:TestPoint_Pad_D1.0mm, F.Cu at (151.3, 57.5)
- added DSDA-4: TestPoint, TestPoint:TestPoint_Pad_D1.0mm, F.Cu at (176.7, 57.5)
- added DSDA-5: TestPoint, TestPoint:TestPoint_Pad_D1.0mm, F.Cu at (115.1, 118.8)
- added DSDA-6: TestPoint, TestPoint:TestPoint_Pad_D1.0mm, F.Cu at (140.5, 118.8)
- added DSDA-7: TestPoint, TestPoint:TestPoint_Pad_D1.0mm, F.Cu at (165.9, 118.8)
- added DSDA-8: TestPoint, TestPoint:TestPoint_Pad_D1.0mm, F.Cu at (191.3, 118.9)
- added J11: Conn_01x04, Connector_JST:JST_GH_BM04B-GHS-TBT_1x04-1MP_P1.25mm_Vertical, F.Cu at (133.2, 101.7)
- added J12: Conn_01x06, Connector_JST:JST_GH_SM06B-GHS-TB_1x06-1MP_P1.25mm_Horizontal, B.Cu at (184.0, 57.1)
- added J15: Conn_01x06, Connector_JST:JST_GH_SM06B-GHS-TB_1x06-1MP_P1.25mm_Horizontal, B.Cu at (133.2, 119.2)
- added J17: Conn_01x04, Connector_JST:JST_GH_BM04B-GHS-TBT_1x04-1MP_P1.25mm_Vertical, F.Cu at (184.0, 101.7)
- added J2: Conn_01x04, Connector_JST:JST_GH_BM04B-GHS-TBT_1x04-1MP_P1.25mm_Vertical, F.Cu at (107.8, 101.7)
- added J20: Conn_01x04, Connector_JST:JST_GH_BM04B-GHS-TBT_1x04-1MP_P1.25mm_Vertical, F.Cu at (158.6, 101.7)
- added J21: Conn_01x06, Connector_JST:JST_GH_SM06B-GHS-TB_1x06-1MP_P1.25mm_Horizontal, B.Cu at (184.0, 119.3)
- added J23: Conn_01x06, Connector_JST:JST_GH_SM06B-GHS-TB_1x06-1MP_P1.25mm_Horizontal, B.Cu at (158.6, 119.2)
- added J4: Conn_01x06, Connector_JST:JST_GH_SM06B-GHS-TB_1x06-1MP_P1.25mm_Horizontal, B.Cu at (107.8, 119.2)
- added J5: Conn_01x04, Connector_JST:JST_GH_BM04B-GHS-TBT_1x04-1MP_P1.25mm_Vertical, F.Cu at (158.6, 74.4)
- added J8: Conn_01x04, Connector_JST:JST_GH_BM04B-GHS-TBT_1x04-1MP_P1.25mm_Vertical, F.Cu at (184.0, 74.4)
- added J9: Conn_01x06, Connector_JST:JST_GH_SM06B-GHS-TB_1x06-1MP_P1.25mm_Horizontal, B.Cu at (158.6, 57.1)
- added R1: 4.7k, Resistor_SMD:R_0603_1608Metric_Pad0.98x0.95mm_HandSolder, F.Cu at (109.3, 114.5)
- added R10: 4.7k, Resistor_SMD:R_0603_1608Metric_Pad0.98x0.95mm_HandSolder, F.Cu at (182.5, 63.4)
- added R11: 120, Resistor_SMD:R_0603_1608Metric_Pad0.98x0.95mm_HandSolder, B.Cu at (101.6, 106.8)
- added R12: 10k, Resistor_SMD:R_0603_1608Metric_Pad0.98x0.95mm_HandSolder, F.Cu at (182.5, 65.0)
- added R13: 600, Resistor_SMD:R_0603_1608Metric_Pad0.98x0.95mm_HandSolder, B.Cu at (103.4, 106.8)
- added R14: 600, Resistor_SMD:R_0603_1608Metric_Pad0.98x0.95mm_HandSolder, B.Cu at (192.0, 69.5)
- added R15: 600, Resistor_SMD:R_0603_1608Metric_Pad0.98x0.95mm_HandSolder, B.Cu at (117.1, 107.0)
- added R16: 4.7k, Resistor_SMD:R_0603_1608Metric_Pad0.98x0.95mm_HandSolder, F.Cu at (157.1, 61.7)
- added R17: 4.7k, Resistor_SMD:R_0603_1608Metric_Pad0.98x0.95mm_HandSolder, F.Cu at (157.1, 63.3)
- added R18: 10k, Resistor_SMD:R_0603_1608Metric_Pad0.98x0.95mm_HandSolder, F.Cu at (157.1, 64.9)
- added R19: 600, Resistor_SMD:R_0603_1608Metric_Pad0.98x0.95mm_HandSolder, B.Cu at (166.6, 69.5)
- added R2: 4.7k, Resistor_SMD:R_0603_1608Metric_Pad0.98x0.95mm_HandSolder, F.Cu at (109.3, 113.0)
- added R20: 120, Resistor_SMD:R_0603_1608Metric_Pad0.98x0.95mm_HandSolder, B.Cu at (164.8, 69.5)
- added R21: 600, Resistor_SMD:R_0603_1608Metric_Pad0.98x0.95mm_HandSolder, B.Cu at (163.0, 69.5)
- added R22: 600, Resistor_SMD:R_0603_1608Metric_Pad0.98x0.95mm_HandSolder, B.Cu at (149.3, 69.3)
- added R23: 120, Resistor_SMD:R_0603_1608Metric_Pad0.98x0.95mm_HandSolder, B.Cu at (151.1, 69.3)
- added R24: 600, Resistor_SMD:R_0603_1608Metric_Pad0.98x0.95mm_HandSolder, B.Cu at (152.9, 69.3)
- added R25: 120, Resistor_SMD:R_0603_1608Metric_Pad0.98x0.95mm_HandSolder, B.Cu at (190.2, 69.5)
- added R26: 600, Resistor_SMD:R_0603_1608Metric_Pad0.98x0.95mm_HandSolder, B.Cu at (188.4, 69.5)
- added R27: 120, Resistor_SMD:R_0603_1608Metric_Pad0.98x0.95mm_HandSolder, B.Cu at (176.5, 69.3)
- added R28: 600, Resistor_SMD:R_0603_1608Metric_Pad0.98x0.95mm_HandSolder, B.Cu at (178.3, 69.3)
- added R29: 4.7k, Resistor_SMD:R_0603_1608Metric_Pad0.98x0.95mm_HandSolder, F.Cu at (134.7, 114.6)
- added R3: 600, Resistor_SMD:R_0603_1608Metric_Pad0.98x0.95mm_HandSolder, B.Cu at (174.7, 69.3)
- added R30: 4.7k, Resistor_SMD:R_0603_1608Metric_Pad0.98x0.95mm_HandSolder, F.Cu at (134.7, 113.0)
- added R31: 10k, Resistor_SMD:R_0603_1608Metric_Pad0.98x0.95mm_HandSolder, F.Cu at (134.7, 111.3)
- added R32: 600, Resistor_SMD:R_0603_1608Metric_Pad0.98x0.95mm_HandSolder, B.Cu at (125.2, 106.8)
- added R33: 120, Resistor_SMD:R_0603_1608Metric_Pad0.98x0.95mm_HandSolder, B.Cu at (127.0, 106.8)
- added R34: 600, Resistor_SMD:R_0603_1608Metric_Pad0.98x0.95mm_HandSolder, B.Cu at (128.8, 106.8)
- added R35: 600, Resistor_SMD:R_0603_1608Metric_Pad0.98x0.95mm_HandSolder, B.Cu at (142.5, 107.0)
- added R36: 120, Resistor_SMD:R_0603_1608Metric_Pad0.98x0.95mm_HandSolder, B.Cu at (140.7, 107.0)
- added R37: 600, Resistor_SMD:R_0603_1608Metric_Pad0.98x0.95mm_HandSolder, B.Cu at (138.9, 107.0)
- added R47: 4.7k, Resistor_SMD:R_0603_1608Metric_Pad0.98x0.95mm_HandSolder, F.Cu at (185.5, 114.6)
- added R48: 4.7k, Resistor_SMD:R_0603_1608Metric_Pad0.98x0.95mm_HandSolder, F.Cu at (185.5, 113.0)
- added R49: 10k, Resistor_SMD:R_0603_1608Metric_Pad0.98x0.95mm_HandSolder, F.Cu at (185.5, 111.4)
- added R50: 600, Resistor_SMD:R_0603_1608Metric_Pad0.98x0.95mm_HandSolder, B.Cu at (176.0, 106.9)
- added R51: 120, Resistor_SMD:R_0603_1608Metric_Pad0.98x0.95mm_HandSolder, B.Cu at (177.8, 106.9)
- added R52: 600, Resistor_SMD:R_0603_1608Metric_Pad0.98x0.95mm_HandSolder, B.Cu at (179.6, 106.9)
- added R53: 600, Resistor_SMD:R_0603_1608Metric_Pad0.98x0.95mm_HandSolder, B.Cu at (193.3, 107.1)
- added R54: 120, Resistor_SMD:R_0603_1608Metric_Pad0.98x0.95mm_HandSolder, B.Cu at (191.5, 107.1)
- added R55: 600, Resistor_SMD:R_0603_1608Metric_Pad0.98x0.95mm_HandSolder, B.Cu at (189.7, 107.1)
- added R56: 4.7k, Resistor_SMD:R_0603_1608Metric_Pad0.98x0.95mm_HandSolder, F.Cu at (160.1, 114.6)
- added R57: 4.7k, Resistor_SMD:R_0603_1608Metric_Pad0.98x0.95mm_HandSolder, F.Cu at (160.1, 113.0)
- added R58: 10k, Resistor_SMD:R_0603_1608Metric_Pad0.98x0.95mm_HandSolder, F.Cu at (160.1, 111.3)
- added R59: 600, Resistor_SMD:R_0603_1608Metric_Pad0.98x0.95mm_HandSolder, B.Cu at (150.6, 106.8)
- added R60: 120, Resistor_SMD:R_0603_1608Metric_Pad0.98x0.95mm_HandSolder, B.Cu at (152.4, 106.8)
- added R61: 600, Resistor_SMD:R_0603_1608Metric_Pad0.98x0.95mm_HandSolder, B.Cu at (154.2, 106.8)
- added R62: 600, Resistor_SMD:R_0603_1608Metric_Pad0.98x0.95mm_HandSolder, B.Cu at (167.9, 107.0)
- added R63: 120, Resistor_SMD:R_0603_1608Metric_Pad0.98x0.95mm_HandSolder, B.Cu at (166.1, 107.0)
- added R64: 600, Resistor_SMD:R_0603_1608Metric_Pad0.98x0.95mm_HandSolder, B.Cu at (164.3, 107.0)
- added R65: 120, Resistor_SMD:R_0603_1608Metric_Pad0.98x0.95mm_HandSolder, B.Cu at (115.3, 107.0)
- added R66: 600, Resistor_SMD:R_0603_1608Metric_Pad0.98x0.95mm_HandSolder, B.Cu at (113.5, 107.0)
- added R7: 10k, Resistor_SMD:R_0603_1608Metric_Pad0.98x0.95mm_HandSolder, F.Cu at (109.3, 111.3)
- added R8: 4.7k, Resistor_SMD:R_0603_1608Metric_Pad0.98x0.95mm_HandSolder, F.Cu at (182.5, 61.8)
- added R9: 600, Resistor_SMD:R_0603_1608Metric_Pad0.98x0.95mm_HandSolder, B.Cu at (99.8, 106.8)
- added SCL3: TestPoint, TestPoint:TestPoint_Pad_D1.0mm, F.Cu at (163.7, 64.8)
- added SCL4: TestPoint, TestPoint:TestPoint_Pad_D1.0mm, F.Cu at (189.0, 64.9)
- added SCL5: TestPoint, TestPoint:TestPoint_Pad_D1.0mm, F.Cu at (102.8, 111.4)
- added SCL6: TestPoint, TestPoint:TestPoint_Pad_D1.0mm, F.Cu at (128.2, 111.5)
- added SCL7: TestPoint, TestPoint:TestPoint_Pad_D1.0mm, F.Cu at (153.6, 111.5)
- added SCL8: TestPoint, TestPoint:TestPoint_Pad_D1.0mm, F.Cu at (178.9, 111.5)
- added SDA3: TestPoint, TestPoint:TestPoint_Pad_D1.0mm, F.Cu at (160.8, 62.9)
- added SDA4: TestPoint, TestPoint:TestPoint_Pad_D1.0mm, F.Cu at (186.1, 62.9)
- added SDA5: TestPoint, TestPoint:TestPoint_Pad_D1.0mm, F.Cu at (105.7, 113.4)
- added SDA6: TestPoint, TestPoint:TestPoint_Pad_D1.0mm, F.Cu at (131.1, 113.4)
- added SDA7: TestPoint, TestPoint:TestPoint_Pad_D1.0mm, F.Cu at (156.4, 113.4)
- added SDA8: TestPoint, TestPoint:TestPoint_Pad_D1.0mm, F.Cu at (181.8, 113.5)
- added U1: PCA9615DP, Package_SO:TSSOP-10_3x3mm_P0.5mm, B.Cu at (108.5, 106.3)
- added U3: PCA9615DP, Package_SO:TSSOP-10_3x3mm_P0.5mm, B.Cu at (157.9, 70.0)
- added U4: PCA9615DP, Package_SO:TSSOP-10_3x3mm_P0.5mm, B.Cu at (183.2, 70.0)
- added U5: PCA9615DP, Package_SO:TSSOP-10_3x3mm_P0.5mm, B.Cu at (133.9, 106.3)
- added U7: PCA9615DP, Package_SO:TSSOP-10_3x3mm_P0.5mm, B.Cu at (184.7, 106.4)
- added U8: PCA9615DP, Package_SO:TSSOP-10_3x3mm_P0.5mm, B.Cu at (159.3, 106.3)
- renumbered REF** to J3
Routing:
- net +5V: track 202.2 -> 605.8 mm, vias 13 -> 37
- net /input5/DSDA+: track 78.5 -> 313.9 mm, vias 2 -> 8
- net /input5/DSCL+: track 74.9 -> 299.6 mm, vias 2 -> 8
- net /input5/DSDA-: track 74.9 -> 299.5 mm, vias 2 -> 8
- net /input5/DSCL-: track 74.8 -> 299.3 mm, vias 2 -> 8
- net +3.3V: track 95.0 -> 264.2 mm, vias 6 -> 18
- net GND: track 120.9 -> 186.8 mm, vias 9 -> 21
- net /scl1: track 44.4 -> 87.2 mm, vias 1 -> 3
- net /sda1: track 51.6 -> 93.3 mm, vias 1 -> 3
- net /scl6: track 2.77 -> 24.2 mm, vias 0 -> 1
- net /scl8: track 51.9 -> 73.3 mm, vias 2 -> 3
- net /scl7: track 33.6 -> 55.0 mm, vias 0 -> 1
- net /scl4: track 24.4 -> 45.8 mm, vias 1 -> 2
- net /sda8: track 58.6 -> 79.4 mm, vias 2 -> 3
- net /sda7: track 43.3 -> 64.1 mm, vias 1 -> 2
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Other:
- board text added: "Input 3"
- board text added: "Input 4"
- board text added: "Input 5"
- board text added: "Input 6"
- board text added: "Input 7"
- board text added: "Input 8"
