File: host/ghost_host.kicad_pcb (KiCad board)
At the start: 2 copper layers, 127.5 x 68.5 mm, 201 parts, among them J1 RGB_3_Pin_Connector, J11 Conn_01x04, J12 Conn_01x06, J14 Conn_01x04, J15 Conn_01x06, J17 Conn_01x04, J18 Conn_01x06, J2 Conn_01x04, J20 Conn_01x04, J21 Conn_01x06, J23 Conn_01x06, J3 Conn_01x04, J4 Conn_01x06, J5 Conn_01x04, J6 Conn_01x06, J8 Conn_01x04, J9 Conn_01x06, U1 PCA9615DP, U2 PCA9615DP, U3 PCA9615DP, U4 PCA9615DP, U5 PCA9615DP, U6 PCA9615DP, U7 PCA9615DP, U8 PCA9615DP, U9 kb2040

Commit message: finish host board v2 layout + production files
Parts:
- removed REF** (x6): TestPoint, TestPoint:TestPoint_Pad_D1.0mm
- removed REF** (x4): 600, Resistor_SMD:R_0603_1608Metric_Pad0.98x0.95mm_HandSolder
- removed REF** (x2): 1u, Capacitor_SMD:C_0603_1608Metric
- removed REF** (x2): 120, Resistor_SMD:R_0603_1608Metric_Pad0.98x0.95mm_HandSolder
- removed REF**: PCA9615DP, Package_SO:TSSOP-10_3x3mm_P0.5mm
- removed REF**: 10uf, Capacitor_SMD:C_0603_1608Metric
- removed REF**: Conn_01x06, Connector_JST:JST_GH_SM06B-GHS-TB_1x06-1MP_P1.25mm_Horizontal
- removed REF** (x2): 4.7k, Resistor_SMD:R_0603_1608Metric_Pad0.98x0.95mm_HandSolder
- removed REF**: 10k, Resistor_SMD:R_0603_1608Metric_Pad0.98x0.95mm_HandSolder
- added G***: LOGO, pcb_footprints:allen_ai, F.Cu at (170.2, 83.8)
- C17, C18, C19, C20, C21, C22, C23, C24: value 10uf -> 10u
- DSCL+1, DSCL+2, DSCL+3, DSCL+4, DSCL+5, DSCL+6, DSCL+7, DSCL+8, DSCL-1, DSCL-2, DSCL-3, DSCL-4, DSCL-5, DSCL-6, DSCL-7, DSCL-8, DSDA+1, DSDA+2, DSDA+3, DSDA+4, DSDA+5, DSDA+6, DSDA+7, DSDA+8, DSDA-1, DSDA-2, DSDA-3, DSDA-4, DSDA-5, DSDA-6, DSDA-7, DSDA-8, SCL1, SCL2, SCL3, SCL4, SCL5, SCL6, SCL7, SCL8, SDA1, SDA2, SDA3, SDA4, SDA5, SDA6, SDA7, SDA8: footprint TestPoint:TestPoint_Pad_D1.0mm -> TestPoint:TestPoint_THTPad_1.0x1.0mm_Drill0.5mm
- moved SCL8 2.25 mm to (180.8, 112.8)
- moved SDA5 2.24 mm to (103.9, 114.8)
- moved SDA6 2.24 mm to (129.3, 114.8)
- moved SDA7 2.24 mm to (154.7, 114.8)
- moved SDA4 2.20 mm to (187.8, 61.5)
- moved SDA2 2.18 mm to (137.0, 61.5)
- moved SDA1 2.16 mm to (111.6, 61.5)
- moved SDA3 2.13 mm to (162.4, 61.5)
- moved SCL2 1.86 mm to (137.0, 63.5)
- moved SCL4 1.84 mm to (187.8, 63.5)
- moved SCL1 1.84 mm to (111.6, 63.5)
- moved SCL3 1.84 mm to (162.4, 63.5)
- moved SCL5 1.77 mm to (103.9, 112.8)
- moved SCL6 1.77 mm to (129.3, 112.8)
- moved SCL7 1.77 mm to (154.7, 112.8)
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Connections:
- DSCL+3 pad 1: /input5/DSCL+ -> /input2/DSCL+
- DSCL+4 pad 1: /input5/DSCL+ -> /input3/DSCL+
- DSCL+5 pad 1: /input5/DSCL+ -> /input/DSCL+
- DSCL+6 pad 1: /input5/DSCL+ -> /input4/DSCL+
- DSCL+7 pad 1: /input5/DSCL+ -> /input7/DSCL+
- DSCL+8 pad 1: /input5/DSCL+ -> /input6/DSCL+
- DSCL-3 pad 1: /input5/DSCL- -> /input2/DSCL-
- DSCL-4 pad 1: /input5/DSCL- -> /input3/DSCL-
- DSCL-5 pad 1: /input5/DSCL- -> /input/DSCL-
- DSCL-6 pad 1: /input5/DSCL- -> /input4/DSCL-
- DSCL-7 pad 1: /input5/DSCL- -> /input7/DSCL-
- DSCL-8 pad 1: /input5/DSCL- -> /input6/DSCL-
- DSDA+3 pad 1: /input5/DSDA+ -> /input2/DSDA+
- DSDA+4 pad 1: /input5/DSDA+ -> /input3/DSDA+
- DSDA+5 pad 1: /input5/DSDA+ -> /input/DSDA+
- DSDA+6 pad 1: /input5/DSDA+ -> /input4/DSDA+
- DSDA+7 pad 1: /input5/DSDA+ -> /input7/DSDA+
- DSDA+8 pad 1: /input5/DSDA+ -> /input6/DSDA+
- DSDA-3 pad 1: /input5/DSDA- -> /input2/DSDA-
- DSDA-4 pad 1: /input5/DSDA- -> /input3/DSDA-
- DSDA-5 pad 1: /input5/DSDA- -> /input/DSDA-
- DSDA-6 pad 1: /input5/DSDA- -> /input4/DSDA-
- DSDA-7 pad 1: /input5/DSDA- -> /input7/DSDA-
- DSDA-8 pad 1: /input5/DSDA- -> /input6/DSDA-
- J11 pad 1: (no net) -> GND
- J11 pad 2: (no net) -> +5V
- J11 pad 3: (no net) -> /sda6
- J11 pad 4: (no net) -> /scl6
- J12 pad 2: /input5/DSDA- -> /input3/DSDA-
- J12 pad 3: /input5/DSDA+ -> /input3/DSDA+
- J12 pad 4: /input5/DSCL+ -> /input3/DSCL+
- J12 pad 5: /input5/DSCL- -> /input3/DSCL-
- J15 pad 2: /input5/DSDA- -> /input4/DSDA-
- J15 pad 3: /input5/DSDA+ -> /input4/DSDA+
- J15 pad 4: /input5/DSCL+ -> /input4/DSCL+
- J15 pad 5: /input5/DSCL- -> /input4/DSCL-
- J17 pad 1: (no net) -> GND
- J17 pad 2: (no net) -> +5V
- J17 pad 3: (no net) -> /sda8
- J17 pad 4: (no net) -> /scl8
- J2 pad 1: (no net) -> GND
- J2 pad 2: (no net) -> +5V
- J2 pad 3: (no net) -> /sda5
- J2 pad 4: (no net) -> /scl5
- J20 pad 1: (no net) -> GND
- J20 pad 2: (no net) -> +5V
- J20 pad 3: (no net) -> /sda7
- J20 pad 4: (no net) -> /scl7
- J21 pad 2: /input5/DSDA- -> /input6/DSDA-
- J21 pad 3: /input5/DSDA+ -> /input6/DSDA+
- J21 pad 4: /input5/DSCL+ -> /input6/DSCL+
- J21 pad 5: /input5/DSCL- -> /input6/DSCL-
- J23 pad 2: /input5/DSDA- -> /input7/DSDA-
- J23 pad 3: /input5/DSDA+ -> /input7/DSDA+
- J23 pad 4: /input5/DSCL+ -> /input7/DSCL+
- J23 pad 5: /input5/DSCL- -> /input7/DSCL-
- J4 pad 2: /input5/DSDA- -> /input/DSDA-
- J4 pad 3: /input5/DSDA+ -> /input/DSDA+
- J4 pad 4: /input5/DSCL+ -> /input/DSCL+
- J4 pad 5: /input5/DSCL- -> /input/DSCL-
- J5 pad 3: /sda3 -> /sda4
- J5 pad 4: /scl3 -> /scl4
- J8 pad 1: (no net) -> GND
- J8 pad 2: (no net) -> +5V
- J8 pad 3: (no net) -> /sda1
- J8 pad 4: (no net) -> /scl1
- J9 pad 2: /input5/DSDA- -> /input2/DSDA-
- J9 pad 3: /input5/DSDA+ -> /input2/DSDA+
- J9 pad 4: /input5/DSCL+ -> /input2/DSCL+
- J9 pad 5: /input5/DSCL- -> /input2/DSCL-
- R1 pad 2: /sda1 -> /sda5
- R11 pad 1: /input5/DSCL+ -> /input/DSCL+
- R11 pad 2: /input5/DSCL- -> /input/DSCL-
- R13 pad 1: /input5/DSCL- -> /input/DSCL-
- R14 pad 2: /input5/DSCL+ -> /input3/DSCL+
- R15 pad 2: /input5/DSDA+ -> /input/DSDA+
- R19 pad 2: /input5/DSCL+ -> /input2/DSCL+
- R2 pad 2: /scl1 -> /scl5
- R20 pad 1: /input5/DSCL+ -> /input2/DSCL+
- R20 pad 2: /input5/DSCL- -> /input2/DSCL-
- R21 pad 1: /input5/DSCL- -> /input2/DSCL-
- R22 pad 2: /input5/DSDA+ -> /input2/DSDA+
- R23 pad 1: /input5/DSDA+ -> /input2/DSDA+
- R23 pad 2: /input5/DSDA- -> /input2/DSDA-
- R24 pad 1: /input5/DSDA- -> /input2/DSDA-
- R25 pad 1: /input5/DSCL+ -> /input3/DSCL+
- R25 pad 2: /input5/DSCL- -> /input3/DSCL-
- R26 pad 1: /input5/DSCL- -> /input3/DSCL-
- R27 pad 1: /input5/DSDA+ -> /input3/DSDA+
- R27 pad 2: /input5/DSDA- -> /input3/DSDA-
- R28 pad 1: /input5/DSDA- -> /input3/DSDA-
- R3 pad 2: /input5/DSDA+ -> /input3/DSDA+
- R32 pad 2: /input5/DSCL+ -> /input4/DSCL+
- R33 pad 1: /input5/DSCL+ -> /input4/DSCL+
- R33 pad 2: /input5/DSCL- -> /input4/DSCL-
- R34 pad 1: /input5/DSCL- -> /input4/DSCL-
- R35 pad 2: /input5/DSDA+ -> /input4/DSDA+
- R36 pad 1: /input5/DSDA+ -> /input4/DSDA+
- R36 pad 2: /input5/DSDA- -> /input4/DSDA-
- R37 pad 1: /input5/DSDA- -> /input4/DSDA-
- R50 pad 2: /input5/DSCL+ -> /input6/DSCL+
- R51 pad 1: /input5/DSCL+ -> /input6/DSCL+
- R51 pad 2: /input5/DSCL- -> /input6/DSCL-
- R52 pad 1: /input5/DSCL- -> /input6/DSCL-
- R53 pad 2: /input5/DSDA+ -> /input6/DSDA+
- R54 pad 1: /input5/DSDA+ -> /input6/DSDA+
- R54 pad 2: /input5/DSDA- -> /input6/DSDA-
- R55 pad 1: /input5/DSDA- -> /input6/DSDA-
- R59 pad 2: /input5/DSCL+ -> /input7/DSCL+
- R60 pad 1: /input5/DSCL+ -> /input7/DSCL+
- R60 pad 2: /input5/DSCL- -> /input7/DSCL-
- R61 pad 1: /input5/DSCL- -> /input7/DSCL-
- R62 pad 2: /input5/DSDA+ -> /input7/DSDA+
- R63 pad 1: /input5/DSDA+ -> /input7/DSDA+
- R63 pad 2: /input5/DSDA- -> /input7/DSDA-
- R64 pad 1: /input5/DSDA- -> /input7/DSDA-
- R65 pad 1: /input5/DSDA+ -> /input/DSDA+
- R65 pad 2: /input5/DSDA- -> /input/DSDA-
- R66 pad 1: /input5/DSDA- -> /input/DSDA-
- R9 pad 2: /input5/DSCL+ -> /input/DSCL+
- SCL5 pad 1: /scl1 -> /scl5
- SDA5 pad 1: /sda1 -> /sda5
- U1 pad 2: /sda1 -> /sda5
- U1 pad 4: /scl1 -> /scl5
- U1 pad 6: /input5/DSCL- -> /input/DSCL-
- U1 pad 7: /input5/DSCL+ -> /input/DSCL+
- U1 pad 8: /input5/DSDA+ -> /input/DSDA+
- U1 pad 9: /input5/DSDA- -> /input/DSDA-
- U3 pad 6: /input5/DSCL- -> /input2/DSCL-
- U3 pad 7: /input5/DSCL+ -> /input2/DSCL+
- U3 pad 8: /input5/DSDA+ -> /input2/DSDA+
- U3 pad 9: /input5/DSDA- -> /input2/DSDA-
- U4 pad 6: /input5/DSCL- -> /input3/DSCL-
- U4 pad 7: /input5/DSCL+ -> /input3/DSCL+
- U4 pad 8: /input5/DSDA+ -> /input3/DSDA+
- U4 pad 9: /input5/DSDA- -> /input3/DSDA-
- U5 pad 6: /input5/DSCL- -> /input4/DSCL-
- U5 pad 7: /input5/DSCL+ -> /input4/DSCL+
- U5 pad 8: /input5/DSDA+ -> /input4/DSDA+
- U5 pad 9: /input5/DSDA- -> /input4/DSDA-
- U7 pad 6: /input5/DSCL- -> /input6/DSCL-
- U7 pad 7: /input5/DSCL+ -> /input6/DSCL+
- U7 pad 8: /input5/DSDA+ -> /input6/DSDA+
- U7 pad 9: /input5/DSDA- -> /input6/DSDA-
- U8 pad 6: /input5/DSCL- -> /input7/DSCL-
- U8 pad 7: /input5/DSCL+ -> /input7/DSCL+
- U8 pad 8: /input5/DSDA+ -> /input7/DSDA+
- U8 pad 9: /input5/DSDA- -> /input7/DSDA-
Routing:
- net +5V: track 605.8 -> 190.0 mm, vias 37 -> 42
- net /input5/DSDA+: track 313.9 -> 39.2 mm, vias 8 -> 1
- net /input5/DSCL+: track 299.6 -> 37.4 mm, vias 8 -> 1
- net /input5/DSDA-: track 299.5 -> 37.4 mm, vias 8 -> 1
- net /input5/DSCL-: track 299.3 -> 37.4 mm, vias 8 -> 1
- net GND: track 186.8 -> 229.4 mm, vias 21 -> 20
- net /input2/DSDA+: track 0.00 -> 39.2 mm, vias 0 -> 1
- net /input3/DSDA+: track 0.00 -> 39.2 mm, vias 0 -> 1
- net /input7/DSDA+: track 0.00 -> 39.2 mm, vias 0 -> 1
- net /input4/DSDA+: track 0.00 -> 39.2 mm, vias 0 -> 1
- net /input/DSDA+: track 0.00 -> 39.2 mm, vias 0 -> 1
- net /input6/DSDA+: track 0.00 -> 39.2 mm, vias 0 -> 1
- net /input7/DSCL+: track 0.00 -> 37.4 mm, vias 0 -> 1
- net /input6/DSCL+: track 0.00 -> 37.4 mm, vias 0 -> 1
- net /input/DSCL+: track 0.00 -> 37.4 mm, vias 0 -> 1
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Other:
- board text added: "IEEE RAS | VEXU GHOST"
- board text added: "INPUT 1 - GPIO 8/9 (2/3) INPUT 2 - GPIO 2/3 (4/5) INPUT 3 - GPIO 4/5 (6/7) INPUT 4 - GPIO 6/7 (8/9) INPUT 5 - GPIO 0/1 (TX/RX) INPUT 6 - GPIO 28/27 (A2/A1) INPUT 7 - GPIO 26/18 (A0/CLK) INPUT 8 - GPIO 20/19 (MI/MO)"
- board text added: "Karmanyaah Malhotra, Andrew Kwa, Gengwen Li, Trung Le, Allen Ai"
- board text removed: "Andrew Kwa et al."
- board text removed: "IEEE RAS-VEX U TEAM GHOST"
- board text removed: "INPUT 1 - GPIO 8/9 INPUT 2 - GPIO 2/3 INPUT 3 - GPIO 4/5 INPUT 4 - GPIO 6/7 INPUT 5 - GPIO 0/1 INPUT 6 - GPIO 28/27 INPUT 7 - GPIO 26/18 INPUT 8 - GPIO 20/19"
