File: color_proximity_imu_breakout/Iteration_2/color/color.kicad_sch (KiCad schematic)
At the start: 13 parts, among them IC2 ISL29125IROZ-T7, J4 Conn_01x05

Commit message: Color Board Iteration 2 Updated
Parts:
- added C1, C2: 10u, Capacitor_SMD:C_0603_1608Metric_Pad1.08x0.95mm_HandSolder, symbol Device:C
- added J1, J2: Conn_01x10, pcb_footprints:GT-B0502MSV27-10S1101, symbol Connector_Generic:Conn_01x10
Connections:
- net +3.3V: now also C1.2, C2.2, J1.9 (Pin_9), J2.9 (Pin_9)
- net +5V: now also J1.10 (Pin_10), J2.10 (Pin_10)
- net GND: now also C1.1, C2.1, J1.6 (Pin_6), J2.6 (Pin_6)
- net scl: now also J1.7 (Pin_7), J2.7 (Pin_7)
- net sda: now also J1.8 (Pin_8), J2.8 (Pin_8)
- no-connect marks 0 -> 10
Other:
- moved on the sheet: C14, J4

Commit message: breakout board iteration 2 updates
Parts:
- removed C14: 10u, Capacitor_SMD:C_0603_1608Metric_Pad1.08x0.95mm_HandSolder, symbol Device:C
- removed J4: Conn_01x05, Connector_PinHeader_2.54mm:PinHeader_1x05_P2.54mm_Vertical, symbol Connector_Generic:Conn_01x05
- removed R30, R32: 120, Resistor_SMD:R_0402_1005Metric, symbol Device:R
- R17, R18: value 120 -> 60
Connections:
- net +3.3V: now also D1.2 (A), D2.2 (A)
- net GND: now also R17.2, R18.2
- removed net +5V: D1.2 (A), D2.2 (A), J1.10 (Pin_10), J2.10 (Pin_10)
- no-connect marks 10 -> 12
Other:
- note removed: "Mark specially on silkscreen"

Commit message: finished base board PCB + created production files for base board and modules
Parts:
- C1, C2: Manufacturer_Name (none) -> Samsung Electro-Mechanics; Manufacturer_Part_Number (none) -> CL10A106KP8NNNC
- C4: Manufacturer_Name (none) -> Samsung Electro-Mechanics; Manufacturer_Part_Number (none) -> CL10B105KB8NQNC
- C5: Manufacturer_Name (none) -> Samsung Electro-Mechanics; Manufacturer_Part_Number (none) -> CL05B104KB54PNC
- D1, D2: Manufacturer_Name (none) -> XINGLIGHT; Manufacturer_Part_Number (none) -> XL-2012UWC-A
- J1, J2: Manufacturer_Name (none) -> G-Switch; Manufacturer_Part_Number (none) -> GT-B0502MSV27-10S1101
Changed lines of the file:
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@@
+			)
+		)
+		(property "Manufacturer_Name" "Samsung Electro-Mechanics"
+			(at 49.53 59.69 0)
+			(effects
+				(font
+					(size 1.27 1.27)
+				)
+				(hide yes)
+			)
+		)
+		(property "Manufacturer_Part_Number" "CL10B105KB8NQNC"
+			(at 49.53 59.69 0)
+			(effects
+				(font
+					(size 1.27 1.27)
+				)
+				(hide yes)
 			)
 		)
@@
 			)
 		)
+		(property "Manufacturer_Name" "G-Switch"
+			(at 69.85 128.27 0)
+			(effects
+				(font
+					(size 1.27 1.27)
+				)
+				(hide yes)
+			)
+		)
+		(property "Manufacturer_Part_Number" "GT-B0502MSV27-10S1101"
+			(at 69.85 128.27 0)
+			(effects
+				(font
+					(size 1.27 1.27)
+				)
+				(hide yes)
+			)
+		)
 		(pin "1"
 		)
@@
 			)
 		)
+		(property "Manufacturer_Name" "Samsung Electro-Mechanics"
+			(at 54.61 59.69 0)
+			(effects
+				(font
+					(size 1.27 1.27)
+				)
+				(hide yes)
+			)
+		)
+		(property "Manufacturer_Part_Number" "CL05B104KB54PNC"
+			(at 54.61 59.69 0)
+			(effects
+				(font
+					(size 1.27 1.27)
+				)
+				(hide yes)
+			)
+		)
 		(pin "2"
 		)
@@
 			)
 		)
+		(property "Manufacturer_Name" "G-Switch"
+			(at 69.85 100.33 0)
+			(effects
+				(font
+					(size 1.27 1.27)
+				)
+				(hide yes)
+			)
+		)
+		(property "Manufacturer_Part_Number" "GT-B0502MSV27-10S1101"
+			(at 69.85 100.33 0)
+			(effects
+				(font
+					(size 1.27 1.27)
+				)
+				(hide yes)
+			)
+		)
 		(pin "1"
 		)
@@
 			)
 		)
+		(property "Manufacturer_Name" "Samsung Electro-Mechanics"
+			(at 53.34 105.41 0)
+			(effects
+				(font
+					(size 1.27 1.27)
+				)
+				(hide yes)
+			)
+		)
+		(property "Manufacturer_Part_Number" "CL10A106KP8NNNC"
+			(at 53.34 105.41 0)
+			(effects
+				(font
+					(size 1.27 1.27)
+				)
+				(hide yes)
+			)
+		)
 		(pin "2"
 		)
@@
 			)
 		)
+		(property "Manufacturer_Name" "XINGLIGHT"
+			(at 119.38 54.61 90)
+			(effects
+				(font
+					(size 1.27 1.27)
+				)
+				(hide yes)
+			)
+		)
+		(property "Manufacturer_Part_Number" "XL-2012UWC-A"
+			(at 119.38 54.61 90)
+			(effects
+				(font
+					(size 1.27 1.27)
+				)
+				(hide yes)
+			)
+		)
 		(pin "2"
 		)
@@
 			)
 		)
+		(property "Manufacturer_Name" "Samsung Electro-Mechanics"
+			(at 53.34 133.35 0)
+			(effects
+				(font
+					(size 1.27 1.27)
+				)
+				(hide yes)
+			)
+		)
+		(property "Manufacturer_Part_Number" "CL10A106KP8NNNC"
+			(at 53.34 133.35 0)
+			(effects
+				(font
+					(size 1.27 1.27)
+				)
+				(hide yes)
+			)
+		)
 		(pin "2"
 		)
@@
 			(at 109.22 54.61 90)
 			(effects
+				(font
+					(size 1.27 1.27)
+				)
+				(hide yes)
+			)
+		)
+		(property "Manufacturer_Name" "XINGLIGHT"
+			(at 109.22 54.61 90)
+			(effects
+				(font
+					(size 1.27 1.27)
+				)
+				(hide yes)
+			)
+		)
+		(property "Manufacturer_Part_Number" "XL-2012UWC-A"
+			(at 109.22 54.61 90)
+			(effects

Commit message: updated production files
Connections:
- net +3.3V: now also C1.1, C2.1, J1.7 (Pin_7), J2.7 (Pin_7); no longer C1.2, C2.2, J1.9 (Pin_9), J2.9 (Pin_9)
- net GND: now also C1.2, C2.2, J1.10 (Pin_10), J2.10 (Pin_10); no longer C1.1, C2.1, J1.6 (Pin_6), J2.6 (Pin_6)
- net scl: now also J1.9 (Pin_9), J2.9 (Pin_9); no longer J1.7 (Pin_7), J2.7 (Pin_7)
Other:
- moved on the sheet: C1, C2
