File: color_proximity_imu_breakout/Iteration_2/proximity/proximity.kicad_sch (KiCad schematic)
At the start: 7 parts, among them IC1 VL53L4CDV0DH_1, J4 Conn_01x05

Commit message: gpio board iteration 2 updated
Parts:
- added C2 (x2): 10u, Capacitor_SMD:C_0603_1608Metric_Pad1.08x0.95mm_HandSolder, symbol Device:C
- added J1, J2: Conn_01x10, pcb_footprints:GT-B0502MSV27-10S1101, symbol Connector_Generic:Conn_01x10
Connections:
- net +3.3V: now also C2.2, C2.2, J1.9 (Pin_9), J2.9 (Pin_9)
- net +5V: now also J1.10 (Pin_10), J2.10 (Pin_10)
- net GND: now also C2.1, C2.1, J1.6 (Pin_6), J2.6 (Pin_6)
- net scl: now also J1.7 (Pin_7), J2.7 (Pin_7)
- net sda: now also J1.8 (Pin_8), J2.8 (Pin_8)
- no-connect marks 1 -> 11

Commit message: finished base board PCB + created production files for base board and modules
Parts:
- removed C1: 10u, Capacitor_SMD:C_0402_1005Metric_Pad0.74x0.62mm_HandSolder, symbol Device:C
- removed J4: Conn_01x05, Connector_PinHeader_2.54mm:PinHeader_1x05_P2.54mm_Vertical, symbol Connector_Generic:Conn_01x05
- C1: renamed from C2; Manufacturer_Name (none) -> Samsung Electro-Mechanics; Manufacturer_Part_Number (none) -> CL10A106KP8NNNC
- C11: Manufacturer_Name (none) -> Samsung Electro-Mechanics; Manufacturer_Part_Number (none) -> CL05B104KB54PNC
- C12: Manufacturer_Name (none) -> Samsung Electro-Mechanics; Manufacturer_Part_Number (none) -> CL10A475KO8NNNC
- C2: Manufacturer_Name (none) -> Samsung Electro-Mechanics; Manufacturer_Part_Number (none) -> CL10A106KP8NNNC
- J1, J2: Manufacturer_Name (none) -> G-Switch; Manufacturer_Part_Number (none) -> GT-B0502MSV27-10S1101

Commit message: updated production files
Connections:
- net +5V is gone; now on net GND: J1.10 (Pin_10), J2.10 (Pin_10)
- net +3.3V: now also C1.1, C2.1, J1.7 (Pin_7), J2.7 (Pin_7); no longer C1.2, C2.2, J1.9 (Pin_9), J2.9 (Pin_9)
- net GND: now also C1.2, C2.2; no longer C1.1, C2.1, J1.6 (Pin_6), J2.6 (Pin_6)
- net scl: now also J1.9 (Pin_9), J2.9 (Pin_9); no longer J1.7 (Pin_7), J2.7 (Pin_7)
- no-connect marks 11 -> 13
Other:
- moved on the sheet: C1, C2
